File: HW/MP3_Player.brd (EAGLE design)
At the start: 100 x 80 mm, 69 parts, among them IC3 ATMEGA8U2, J1 ISP/SPI, Q1 12.288MHz, U1 3.3V, U3 VS1053, U4 1.8V, U5 MCP73831, U6 USD-SOCKET, X2 USBSMD, Y2 8Mhz

Commit message: changed buttons, oscillator and JST connector
Parts:
- removed IC3: ATMEGA8U2, hf:TQFP32-08
- removed LCD3: UG-2832HSWEG04, microbuilder:UG-2832HSWEG04_WRAPAROUND
- removed Y2: 8Mhz, SparkFun-FreqCtrl:HC49UP
- added C18, C19: 0.1uF, SparkFun-Capacitors:0603-CAP
- added C20: 0.1uF, rcl:C0603K
- added OLED1: UG-2832HSWEG04, microbuilder:UG-2832HSWEG04_WRAPAROUND
- added Q2: 12.288MHz, SparkFun:CRYSTAL-SMD-5X3
- added U2: 1.8V, SparkFun-PowerIC:SC70
- C10, C11, C12, C13, C14, C15, C16, C2, C3, C4, C5, C8: device SparkFun-Capacitors:0603-CAP -> rcl:C0603K
- C23, C24: value 20p -> 18p
- C7: device rcl:C0402 -> rcl:C0603K
- J2: value (none) -> LIPO-BATTERY-CONNECTOR; device SparkFun-Connectors:JST-2-SMD -> pero_library:JST-LIPO-CONNECTOR-1.25MM
- Q1: value 12.288MHz -> (none); device SparkFun:CRYSTAL-SMD-5X3 -> pero_library:6X3.2MM
- S1: value SWITCH-SMD -> Reset; device SparkFun:TACTILE_SWITCH_SMD -> pero_library:TACTILE-SWITCH-SKSGAAE010
- S2: value PLAY/PAUSE -> Play/Pause; device SparkFun:TACTILE_SWITCH_SMD -> pero_library:TACTILE-SWITCH-SKSGAAE010
- S3: device SparkFun:TACTILE_SWITCH_SMD -> pero_library:TACTILE-SWITCH-SKSGAAE010
- S4: value BACK -> BCK; device SparkFun:TACTILE_SWITCH_SMD -> pero_library:TACTILE-SWITCH-SKSGAAE010
- S5: value SWITCH-SMD -> (none); device SparkFun:TACTILE_SWITCH_SMD -> pero_library:TACTILE-SWITCH-SKSGAAE010
- U3: value VS1053 -> ATMEGA32U2; device SparkFun-DigitalIC:LQFP-48 -> hf:TQFP32-08
- U4: value 1.8V -> VS1053; device SparkFun-PowerIC:SC70 -> SparkFun-DigitalIC:LQFP-48
- moved R16 302.0 mm to (90.2, 54.6), turned to 90 degrees
- moved C33 300.0 mm to (118.1, 73.7)
- moved C34 300.0 mm to (124.5, 73.7)
- moved C35 300.0 mm to (130.8, 73.7)
- moved C36 300.0 mm to (118.1, 71.1)
- moved C37 300.0 mm to (124.5, 71.1)
- moved C38 300.0 mm to (130.8, 71.1)
- moved R11 300.0 mm to (118.1, 68.6)
- moved R15 296.7 mm to (86.4, 54.6), turned to 90 degrees
- moved R14 291.3 mm to (82.5, 54.6), turned to 90 degrees
- moved R10 286.0 mm to (78.7, 54.6), turned to 90 degrees
- moved S5 235.3 mm to (62.2, 10.2), turned to 270 degrees
- moved S4 234.7 mm to (68.6, 10.2), turned to 270 degrees
- moved S2 234.5 mm to (81.3, 10.2), turned to 270 degrees
- moved S3 234.4 mm to (74.9, 10.2), turned to 270 degrees
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Connections:
- new net 3.3V1: C20.1
- new net OLED-DC: OLED1.10, U3.20
- net 1.8V: now also U2.5, U4.24, U4.31, U4.7; no longer U3.24, U3.31, U3.5, U3.7
- net 3.3V: now also C18.1, C19.1, OLED1.5, OLED1.7, S2.P$2, S3.P$2, S4.P$2, S5.P$2, U2.1, U2.3, U3.31, U3.4, U4.14, U4.19, U4.32, U4.38, U4.43, U4.45, U4.6; no longer IC3.31, IC3.32, IC3.4, LCD3.5, LCD3.7, S2.3, S3.3, S4.3, S5.3, U3.14, U3.19, U3.38, U3.43, U3.45, U3.6, U4.1, U4.3
- net G1: now also U4.10, U4.11, U4.12, U4.9; no longer U3.10, U3.11, U3.12, U3.9
- net G2: now also U4.25; no longer U3.25
- net GBUF: now also U4.42; no longer U3.42
- net GND: now also C18.2, C19.2, C20.2, J2.P$2, OLED1.6, S1.P$1, U2.2, U3.28, U3.3, U4.16, U4.20, U4.21, U4.22, U4.33, U4.34, U4.35, U4.37, U4.4, U4.40, U4.41, U4.47; no longer IC3.28, IC3.3, J2.1, LCD3.6, S1.1, U3.16, U3.20, U3.21, U3.22, U3.33, U3.34, U3.35, U3.37, U3.4, U3.40, U3.41, U3.47, U4.2
- net GPIO4: now also U4.36; no longer U3.36
- net LEFT: now also U4.46; no longer U3.46
- net MIDI-RX: now also U4.26; no longer U3.26
- net MISO: now also U3.17, U4.30; no longer IC3.17, LCD3.10, U3.30
- net MOSI: now also OLED1.12, U3.16, U4.29; no longer IC3.16, LCD3.12, U3.29
- net MP3-CS: now also U4.23; no longer U3.23
- net MP3-DCS: now also U4.13; no longer U3.13
- net MP3-DREQ: now also U4.8; no longer U3.8
- net MP3-RST: now also U4.3; no longer U3.3
- net N$1: now also U3.12; no longer IC3.12
- net N$10: now also Q2.1, U4.17; no longer Q1.1, U3.17
- net N$11: now also U3.18; no longer IC3.18
- net N$12: now also U3.8; no longer IC3.8
- net N$18: now also S2.P$1, U3.26; no longer IC3.5, S2.1
- net N$19: now also S3.P$1, U3.25; no longer IC3.26, S3.1
- net N$20: now also Q1.P$2, U3.1; no longer IC3.1, Y2.2
- net N$21: now also Q1.P$1, U3.2; no longer IC3.2, Y2.1
- net N$22: now also U3.29; no longer IC3.29
- net N$23: now also U3.30; no longer IC3.30
- net N$27: now also S4.P$1, U3.23; no longer IC3.25, S4.1
- net N$28: now also S5.P$1, U3.22; no longer IC3.23, S5.1
- net N$29: now also OLED1.11; no longer LCD3.11
- net N$30: now also U3.19; no longer IC3.19
- net N$44: now also OLED1.2; no longer LCD3.2
- net N$45: now also OLED1.1; no longer LCD3.1
- net N$46: now also OLED1.4; no longer LCD3.4
- net N$47: now also OLED1.3; no longer LCD3.3
- net N$48: now also OLED1.13; no longer LCD3.13
- net N$49: now also OLED1.14; no longer LCD3.14
- net N$55: now also OLED1.15; no longer LCD3.15
- net N$7: now also U3.13; no longer IC3.13
- net N$9: now also Q2.3, U4.18; no longer Q1.3, U3.18
- net OLED-CS: now also OLED1.8; no longer LCD3.8
- net OLED-RST: now also OLED1.9; no longer LCD3.9
- net RCAP: now also U4.44; no longer U3.44
- net RIGHT: now also U4.39; no longer U3.39
- net RST: now also S1.P$2, U3.24; no longer IC3.24, S1.3
- net SCK: now also U3.15, U4.28; no longer IC3.15, U3.28
- net SS: now also U3.14; no longer IC3.14
- net VBAT: now also J2.P$1; no longer J2.2
- net VCC: now also U3.27; no longer IC3.27
Routing:
- net VBATT: track 0.00 -> 9.46 mm
Other:
- board size 100 x 80 mm -> 160 x 20 mm

Commit message: Changed uSD socket. Components placed
Parts:
- removed LED3: Power, SparkFun:LED-0603
- removed R12: 100k, SparkFun-Resistors:0603-RES
- removed R25: 1k, SparkFun:0402-RES
- removed U6: USD-SOCKET, SparkFun:MICRO-SD-SOCKET-PP
- added C21, C25: (no value), SparkFun-Capacitors:EIA3216
- added J3: USD-SDIO-SOCKETJLH, pero_library:DM3AT-SF-PEJM5
- added JP2, JP3, JP4: (no value), SparkFun-Passives:PAD-JUMPER-3-2OF3_NC_BY_TRACE_YES_SILK_FULL_BOX
- added LED2: RED, SparkFun-LED:LED-0603
- added R18: 330, rcl:R0603
- C10, C11, C12, C13, C14, C15, C20, C3, C4, C5, C8: device rcl:C0603K -> rcl:C0603
- C19, C9: device SparkFun-Capacitors:0603-CAP -> rcl:C0603
- F2: value PTCSMD -> PTC0603; device SparkFun:PTC-1206 -> SparkFun-PowerIC:0603
- LED1: value Power -> RED
- R1, R2, R3, R4, R5, R6, R7, R8, R9: device SparkFun-Resistors:0603-RES -> rcl:R0603
- R10, R14, R15, R16, R17: device SparkFun:0402-RES -> rcl:R0603
- S5: value (none) -> Reserved
- U1: value 3.3V -> 3.3V/150mA
- U2: value 1.8V -> 1.8V/100mA
- U4: value VS1053 -> VS1053B
- moved D2 180.2 mm to (148.7, 2.54), turned to 90 degrees
- moved C17 179.6 mm to (146.9, 16.4), turned to 270 degrees
- moved J2 176.6 mm to (138.0, 13.0), turned to 180 degrees
- moved R13 176.0 mm to (143.1, 17.7), turned to 0 degrees
- moved U5 174.0 mm to (143.1, 15.1), turned to 270 degrees
- moved C7 171.9 mm to (142.7, 12.7), turned to 180 degrees
- moved U1 171.5 mm to (144.8, 2.54), turned to 90 degrees
- moved S1 170.4 mm to (135.8, 5.84), turned to 180 degrees
- moved D1 169.9 mm to (142.2, 10.8), turned to 180 degrees
- moved C4 167.7 mm to (144.4, 4.95)
- moved X2 162.7 mm to (153.7, 10.2)
- moved C5 162.6 mm to (138.6, 2.92), turned to 90 degrees
- moved C6 162.1 mm to (140.7, 2.67), turned to 270 degrees
- moved R17 139.0 mm to (135.3, 1.40), turned to 180 degrees
- moved F2 133.5 mm to (148.6, 6.35), turned to 270 degrees
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Connections:
- net VBATT renamed VIN
- removed net 3.3V1: C20.1
- removed net D-1: R24.1
- removed net D-2: X2.D-
- removed net GPIO4: R12.2, U4.36
- new net 3.3V2: R18.2, U3.6
- new net N$17: R24.1, X2.D-
- new net PWM_L: C21.A, U3.23
- new net PWM_LEFT: R16.2, S5.P$1, S5.P$3, U3.11
- new net PWM_R: C25.A, U3.25
- net 3.3V: now also C20.1, J3.P$4, S2.P$4, S3.P$4, S4.P$4, S5.P$4; no longer U6.4
- net G2: now also U4.33, U4.34, U4.36
- net GBUF: now also JP4.1, JP4.2
- net GND: now also J3.P$10, J3.P$11, J3.P$12, J3.P$13, J3.P$14, J3.P$6, J3.P$9, JP4.3, LED2.C, S1.P$3; no longer LED3.C, R12.1, U4.33, U4.34, U6.6, U6.CD1, U6.CD2, U6.GND1, U6.GND3
- net LEFT: now also JP2.1
- net MISO: now also J3.P$7; no longer U6.7
- net MOSI: now also J3.P$3; no longer U6.3
- net N$12: now also U3.7; no longer U3.8
- net N$14: now also JP2.2
- net N$18: now also S2.P$3, U3.8; no longer U3.26
- net N$19: now also S3.P$3, U3.9; no longer U3.25
- net N$25: now also C21.C, JP2.3; no longer LED3.A, R25.1
- net N$27: now also S4.P$3, U3.10; no longer U3.23
- net N$28: now also C25.C, JP3.3; no longer R16.2, S5.P$1, U3.22
- net N$8: now also LED2.A, R18.1; no longer C17.A, D2.A, U5.4
- net RIGHT: now also JP3.1, JP3.2
- net RST: now also S1.P$4
- net SCK: now also J3.P$5; no longer U6.5
- net SD-CS: now also J3.P$2; no longer U6.2
- net VUSB: now also C17.A, D2.A, U5.4; no longer R25.2
Routing:
- net VIN: track 9.46 -> 0.00 mm

Commit message: Comit before 1st autorouter
Parts:
- moved C23 0.28 mm to (132.5, 16.4)
- moved C24 0.13 mm to (129.3, 16.4)
Changed lines of the file:
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@@
 </class>
 </classes>
-<designrules name="default">
+<designrules name="default *">
 <description language="de">&lt;b&gt;EAGLE Design Rules&lt;/b&gt;
 &lt;p&gt;
@@
 <param name="mtCopper" value="0.035mm 0.035mm 0.035mm 0.035mm 0.035mm 0.035mm 0.035mm 0.035mm 0.035mm 0.035mm 0.035mm 0.035mm 0.035mm 0.035mm 0.035mm 0.035mm"/>
 <param name="mtIsolate" value="1.5mm 0.15mm 0.2mm 0.15mm 0.2mm 0.15mm 0.2mm 0.15mm 0.2mm 0.15mm 0.2mm 0.15mm 0.2mm 0.15mm 0.2mm"/>
-<param name="mdWireWire" value="8mil"/>
-<param name="mdWirePad" value="8mil"/>
-<param name="mdWireVia" value="8mil"/>
-<param name="mdPadPad" value="8mil"/>
-<param name="mdPadVia" value="8mil"/>
-<param name="mdViaVia" value="8mil"/>
+<param name="mdWireWire" value="10mil"/>
+<param name="mdWirePad" value="10mil"/>
+<param name="mdWireVia" value="10mil"/>
+<param name="mdPadPad" value="2mil"/>
+<param name="mdPadVia" value="10mil"/>
+<param name="mdViaVia" value="10mil"/>
 <param name="mdSmdPad" value="8mil"/>
 <param name="mdSmdVia" value="8mil"/>
-<param name="mdSmdSmd" value="8mil"/>
+<param name="mdSmdSmd" value="2mil"/>
 <param name="mdViaViaSameLayer" value="8mil"/>
 <param name="mnLayersViaInSmd" value="2"/>
-<param name="mdCopperDimension" value="40mil"/>
-<param name="mdDrill" value="8mil"/>
+<param name="mdCopperDimension" value="0mil"/>
+<param name="mdDrill" value="10mil"/>
 <param name="mdSmdStop" value="0mil"/>
 <param name="msWidth" value="10mil"/>
@@
 <element name="U3" library="hf" package="TQFP32-08" value="ATMEGA32U2" x="128.27" y="6.35" rot="R270"/>
 <element name="C22" library="rcl" package="C0603" value="1u" x="135.255" y="3.429"/>
-<element name="C23" library="rcl" package="C0603" value="18p" x="132.207" y="16.256"/>
-<element name="C24" library="rcl" package="C0603" value="18p" x="129.286" y="16.256" rot="R180"/>
+<element name="C23" library="rcl" package="C0603" value="18p" x="132.461" y="16.383"/>
+<element name="C24" library="rcl" package="C0603" value="18p" x="129.286" y="16.383" rot="R180"/>
 <element name="R23" library="rcl" package="R0603" value="22" x="148.082" y="9.398" rot="R180"/>
 <element name="R24" library="rcl" package="R0603" value="22" x="148.082" y="11.557" rot="R180"/>
@@
 <wire x1="137.414" y1="12.065" x2="141.8289" y2="15.113" width="0" layer="19" extent="1-16"/>
 <wire x1="141.873" y1="12.7" x2="141.8289" y2="15.113" width="0" layer="19" extent="1-1"/>
-<wire x1="131.357" y1="16.256" x2="137.414" y2="12.065" width="0" layer="19" extent="1-16"/>
-<wire x1="130.136" y1="16.256" x2="131.357" y2="16.256" width="0" layer="19" extent="1-1"/>
-<wire x1="126.48" y1="16.256" x2="130.136" y2="16.256" width="0" layer="19" extent="1-1"/>
+<wire x1="131.611" y1="16.383" x2="137.414" y2="12.065" width="0" layer="19" extent="1-16"/>
+<wire x1="130.136" y1="16.383" x2="131.611" y2="16.383" width="0" layer="19" extent="1-1"/>
+<wire x1="126.48" y1="16.256" x2="130.136" y2="16.383" width="0" layer="19" extent="1-1"/>
 <wire x1="126.619" y1="14.058" x2="126.48" y2="16.256" width="0" layer="19" extent="1-1"/>
 <wire x1="129.47" y1="10.6426" x2="126.619" y2="14.058" width="0" layer="19" extent="1-1"/>
@@
 <contactref element="C23" pad="2"/>
 <contactref element="Q1" pad="P$2"/>
-<wire x1="131.07" y1="10.6426" x2="133.057" y2="16.256" width="0" layer="19" extent="1-1"/>
+<wire x1="131.07" y1="10.6426" x2="133.311" y2="16.383" width="0" layer="19" extent="1-1"/>
 <wire x1="132.883" y1="13.462" x2="131.07" y2="10.6426" width="0" layer="19" extent="1-1"/>
 </signal>
@@
 <contactref element="C24" pad="2"/>
 <contactref element="Q1" pad="P$1"/>
-<wire x1="130.27" y1="10.6426" x2="128.436" y2="16.256" width="0" layer="19" extent="1-1"/>
+<wire x1="130.27" y1="10.6426" x2="128.436" y2="16.383" width="0" layer="19" extent="1-1"/>
 <wire x1="128.483" y1="13.462" x2="130.27" y2="10.6426" width="0" layer="19" extent="1-1"/>
 </signal>
@@
 </signal>
 </signals>
+<errors>
+</errors>
 </board>
 </drawing>

Commit message: Micro USB instead of mini USB. Created "No MP3" variant. Audio jack verified.
Parts:
- removed X2: USBSMD, SparkFun:USB-MINIB
- added J4: (no value), SparkFun-Connectors:USB-B-MICRO-SMD_V03
- moved R24 3.77 mm to (150.7, 8.89)
- moved R23 3.14 mm to (150.7, 11.0)
Connections:
- net GND: no longer X2.GND
- net N$17: now also J4.D-; no longer X2.D-
- net N$24: now also J4.VBUS; no longer X2.VBUS
- net N$26: now also J4.D+; no longer X2.D+
Routing:
- added copper zone on layer 1, net GND
- added copper zone on layer 16, net GND

Commit message: added 3d model. new button.
Parts:
- removed J1: ISP/SPI, SparkFun:2X3
- removed LED1: RED, SparkFun-LED:LED-0603
- added S6: Vol Down, pero_library:TACTILE-SWITCH-SKSGAAE010
- C16, C2: device rcl:C0603K -> rcl:C0603
- C18: device SparkFun-Capacitors:0603-CAP -> rcl:C0603
- R8: value 330 -> 10k
- S5: value Reserved -> Vol Up
- moved R8 151.9 mm to (10.0, -40.0)
- moved C6 53.9 mm to (194.7, 2.92), turned to 90 degrees
- moved F2 53.8 mm to (202.3, 3.41), turned to 180 degrees
- moved D2 53.8 mm to (202.5, 1.28), turned to 0 degrees
- moved C4 53.4 mm to (197.8, 4.49)
- moved U1 53.3 mm to (198.1, 1.83)
- moved C5 53.2 mm to (191.7, 2.03), turned to 270 degrees
- moved R23 51.1 mm to (201.8, 7.92)
- moved R24 51.1 mm to (201.8, 5.76)
- moved C17 50.8 mm to (197.0, 7.57), turned to 180 degrees
- moved C23 50.4 mm to (182.8, 16.0)
- moved C24 50.4 mm to (179.7, 16.0)
- moved Q1 50.4 mm to (181.1, 13.1)
- moved J4 50.2 mm to (208.0, 6.00)
- moved LED2 50.0 mm to (175.6, 15.3)
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Connections:
- removed net 5V-MOSI: J1.4
- removed net 5V-SCK: J1.3
- net 3.3V: now also S6.P$2, S6.P$4; no longer R8.2
- net GND: now also R8.1; no longer J1.6, LED1.C
- net MISO: no longer J1.1
- net N$1: now also U3.21; no longer U3.12
- net N$6: now also R8.2, S6.P$1, S6.P$3, U3.12; no longer LED1.A, R8.1
- net VCC: no longer J1.2
Routing:
- net 3.3V: track 0.00 -> 260.7 mm, vias 0 -> 5
- net PWM_L: track 0.00 -> 185.0 mm, vias 0 -> 4
- net PWM_R: track 0.00 -> 163.7 mm, vias 0 -> 2
- net MOSI: track 0.00 -> 133.8 mm, vias 0 -> 2
- net OLED-DC: track 0.00 -> 129.0 mm, vias 0 -> 2
- net N$18: track 0.00 -> 35.9 mm
- net 1.8V: track 0.00 -> 33.7 mm
- net N$22: track 0.00 -> 30.9 mm, vias 0 -> 2
- net RIGHT: track 0.00 -> 28.5 mm, vias 0 -> 1
- net SCK: track 0.00 -> 27.9 mm, vias 0 -> 2
- net N$23: track 0.00 -> 26.1 mm
- net MISO: track 0.00 -> 25.7 mm, vias 0 -> 2
- net N$27: track 0.00 -> 24.3 mm, vias 0 -> 3
- net VIN: track 0.00 -> 22.9 mm, vias 0 -> 2
- net GND: track 0.00 -> 21.5 mm, vias 0 -> 11
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Other:
- board size 160 x 20 mm -> 210 x 17 mm

Commit message: Auto router not bad
Parts:
- moved R8 89.9 mm to (86.1, 7.97), flipped to the bottom, turned to 270 degrees
- moved S6 85.0 mm to (86.0, 8.00), turned to 90 degrees
- moved S5 78.5 mm to (91.0, 8.00), turned to 270 degrees
- moved R10 74.1 mm to (91.1, 7.97), flipped to the bottom, turned to 270 degrees
- moved S3 73.4 mm to (96.0, 8.00), turned to 90 degrees
- moved R14 71.2 mm to (96.0, 7.97), flipped to the bottom, turned to 270 degrees
- moved R15 68.3 mm to (101.0, 8.03), flipped to the bottom
- moved R16 65.3 mm to (106.0, 7.97), flipped to the bottom, turned to 270 degrees
- moved S4 60.9 mm to (101.0, 8.00), turned to 90 degrees
- moved S2 55.8 mm to (106.0, 8.00), turned to 90 degrees
- moved J3 8.06 mm to (147.4, 14.5)
- moved LED2 6.43 mm to (169.7, 12.6), turned to 0 degrees
- moved C18 4.77 mm to (172.0, 14.0), turned to 180 degrees
- moved C24 4.02 mm to (177.0, 13.0), turned to 270 degrees
- moved R3 3.90 mm to (32.0, 11.0), flipped to the bottom, turned to 0 degrees
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Connections:
- net PWM_LEFT: no longer S5.P$1, S5.P$3
Routing:
- net N$6: track 0.00 -> 103.4 mm, vias 0 -> 3
- net 3.3V: track 260.7 -> 344.3 mm, vias 5 -> 6
- net N$19: track 11.5 -> 88.4 mm, vias 0 -> 3
- net N$18: track 35.9 -> 103.7 mm, vias 0 -> 2
- net N$27: track 24.3 -> 82.1 mm
- net PWM_LEFT: track 16.5 -> 67.9 mm, vias 2 -> 1
- net MOSI: track 133.8 -> 154.4 mm, vias 2 -> 4
- net N$49: track 0.00 -> 15.6 mm, vias 0 -> 2
- net GND: track 21.5 -> 7.08 mm, vias 11 -> 12
- net RIGHT: track 28.5 -> 15.5 mm
- net 1.8V: track 33.7 -> 44.2 mm
- net OLED-DC: track 129.0 -> 138.3 mm, vias 2 -> 0
- net PWM_L: track 185.0 -> 177.0 mm, vias 4 -> 2
- net MIDI-RX: track 0.00 -> 7.14 mm, vias 0 -> 2
- net MISO: track 25.7 -> 32.7 mm
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Other:
- board size 210 x 17 mm -> 210 x 15 mm

Commit message: completed routing, now just checking
Routing:
- net MISO: track 32.7 -> 179.0 mm, vias 2 -> 5
- net SCK: track 28.4 -> 171.3 mm, vias 2 -> 3
- net GBUF: track 6.48 -> 38.1 mm, vias 1 -> 3
- net LEFT: track 4.63 -> 32.0 mm, vias 1 -> 2
- net 3.3V: track 344.3 -> 368.6 mm, vias 6 -> 8
- net RIGHT: track 15.5 -> 35.2 mm, vias 1 -> 5
- net N$9: track 4.38 -> 17.5 mm, vias 0 -> 2
- net GND: track 7.08 -> 20.0 mm, vias 12 -> 37
- net N$10: track 8.46 -> 18.3 mm, vias 0 -> 2
- net MP3-RST: track 0.00 -> 8.85 mm, vias 0 -> 1
- net RCAP: track 0.00 -> 4.33 mm, vias 0 -> 1
- net MIDI-RX: track 7.14 -> 4.61 mm
- net 1.8V: track 44.2 -> 46.6 mm
- net G2: track 13.4 -> 14.6 mm, vias 0 -> 2
- net PWM_R: track 161.9 -> 162.9 mm
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
Commit message: Completed routing and verified. Added RC filters
Parts:
- added C26, C27: 0.1uF, rcl:C0603
- added R12, R19: 68, rcl:R0603
- C21, C25: value (none) -> 10uF
- moved C25 1.15 mm to (22.4, 13.8)
- moved C8 0.10 mm to (25.1, 11.0)
- moved C9 0.10 mm to (40.1, 11.0)
- moved C3 0.05 mm to (25.1, 4.00)
- moved R1 0.05 mm to (25.1, 7.00)
- moved R18 0.05 mm to (172.0, 11.9)
Connections:
- net RCAP renamed N$33
- new net N$13: JP1.SLEEVE, JP4.2
- new net N$31: JP1.RING, JP3.2
- new net N$32: C21.A, C26.1, R12.1
- new net PWM_L1: C25.A, C27.1, R19.1
- net GBUF: no longer JP1.SLEEVE, JP4.2
- net GND: now also C26.2, C27.2
- net PWM_L: now also R12.2; no longer C21.A
- net PWM_R: now also R19.2; no longer C25.A
- net RIGHT: no longer JP1.RING, JP3.2
Routing:
- net RIGHT: track 35.2 -> 20.3 mm, vias 5 -> 4
- net N$31: track 0.00 -> 14.3 mm, vias 0 -> 1
- net N$14: track 11.5 -> 4.37 mm
- net N$13: track 0.00 -> 4.19 mm, vias 0 -> 1
- net GBUF: track 38.1 -> 42.1 mm
- net PWM_L1: track 0.00 -> 3.63 mm, vias 0 -> 1
- net N$32: track 0.00 -> 2.73 mm, vias 0 -> 1
- net PWM_R: track 162.9 -> 160.3 mm
- net N$4: track 4.74 -> 2.75 mm
- net N$28: track 3.74 -> 2.59 mm
- net PWM_L: track 177.0 -> 178.2 mm
- net N$46: track 19.6 -> 20.7 mm
- net N$48: track 9.64 -> 10.7 mm
- net N$55: track 11.1 -> 11.6 mm
- net GND: track 20.0 -> 19.8 mm, vias 37 -> 65
Other:
- board size 210 x 15 mm -> 210.9 x 16 mm
