File: HW/MP3_Player.brd (EAGLE design)
At the start: 210.9 x 16 mm, 79 parts, among them J2 LIPO-BATTERY-CONNECTOR, J3 USD-SDIO-SOCKETJLH, Q2 12.288MHz, U1 3.3V/150mA, U2 1.8V/100mA, U3 ATMEGA32U2, U4 VS1053B, U5 MCP73831

Commit message: gerber files generated
Other:
- board size 210.9 x 16 mm -> 210 x 15 mm
Changed lines of the file:
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@@
 <layer number="15" name="Route15" color="4" fill="6" visible="no" active="no"/>
 <layer number="16" name="Bottom" color="1" fill="1" visible="yes" active="yes"/>
-<layer number="17" name="Pads" color="2" fill="1" visible="yes" active="yes"/>
-<layer number="18" name="Vias" color="2" fill="1" visible="yes" active="yes"/>
-<layer number="19" name="Unrouted" color="6" fill="1" visible="yes" active="yes"/>
+<layer number="17" name="Pads" color="2" fill="1" visible="no" active="yes"/>
+<layer number="18" name="Vias" color="2" fill="1" visible="no" active="yes"/>
+<layer number="19" name="Unrouted" color="6" fill="1" visible="no" active="yes"/>
 <layer number="20" name="Dimension" color="15" fill="1" visible="yes" active="yes"/>
-<layer number="21" name="tPlace" color="7" fill="1" visible="yes" active="yes"/>
-<layer number="22" name="bPlace" color="7" fill="1" visible="yes" active="yes"/>
+<layer number="21" name="tPlace" color="7" fill="1" visible="no" active="yes"/>
+<layer number="22" name="bPlace" color="7" fill="1" visible="no" active="yes"/>
 <layer number="23" name="tOrigins" color="15" fill="1" visible="no" active="yes"/>
 <layer number="24" name="bOrigins" color="15" fill="1" visible="no" active="yes"/>
@@
 <description>Music player za ugradnju u hrbat knjige.</description>
 <plain>
-<wire x1="-0.4" y1="-0.5" x2="210.5" y2="-0.4" width="0" layer="20"/>
-<wire x1="210.5" y1="-0.4" x2="210.5" y2="15.5" width="0" layer="20"/>
-<wire x1="210.5" y1="15.5" x2="-0.4" y2="15.4" width="0" layer="20"/>
-<wire x1="-0.4" y1="15.4" x2="-0.4" y2="-0.5" width="0" layer="20"/>
+<wire x1="0" y1="0" x2="210" y2="0" width="0" layer="20"/>
+<wire x1="210" y1="0" x2="210" y2="15" width="0" layer="20"/>
+<wire x1="210" y1="15" x2="0" y2="15" width="0" layer="20"/>
+<wire x1="0" y1="15" x2="0" y2="0" width="0" layer="20"/>
 <wire x1="210" y1="0" x2="0" y2="0" width="0" layer="39"/>
-<dimension x1="0" y1="20" x2="210" y2="22" x3="105" y3="21" textsize="1.778" layer="20" dtype="horizontal" visible="yes"/>
-<dimension x1="86" y1="8" x2="91" y2="8" x3="88.5" y3="-9" textsize="1.27" layer="20" dtype="horizontal" extwidth="0.1" extlength="1" extoffset="8" precision="0" visible="yes"/>
-<dimension x1="91" y1="8" x2="96" y2="8" x3="93.5" y3="-9" textsize="1.27" layer="20" dtype="horizontal" extwidth="0.1" extlength="1" extoffset="8" precision="0" visible="yes"/>
-<dimension x1="96" y1="8" x2="101" y2="8" x3="98.5" y3="-9" textsize="1.27" layer="20" dtype="horizontal" extwidth="0.1" extlength="1" extoffset="8" precision="0" visible="yes"/>
-<dimension x1="101" y1="8" x2="106" y2="8" x3="103.5" y3="-9" textsize="1.27" layer="20" dtype="horizontal" extwidth="0.1" extlength="1" extoffset="8" precision="0" visible="yes"/>
-<dimension x1="50" y1="-10" x2="80" y2="-10" x3="65" y3="-7" textsize="1.27" layer="20" visible="yes"/>
-<dimension x1="0" y1="15" x2="0" y2="0" x3="-4" y3="7.5" textsize="1.27" layer="20" visible="yes"/>
-<dimension x1="0" y1="0" x2="50" y2="0" x3="25" y3="-7" textsize="1.27" layer="20" extoffset="3" visible="yes"/>
+<dimension x1="0" y1="20" x2="210" y2="22" x3="105" y3="21" textsize="1.778" layer="51" dtype="horizontal" visible="yes"/>
+<dimension x1="86" y1="8" x2="91" y2="8" x3="88.5" y3="-9" textsize="1.27" layer="51" dtype="horizontal" extwidth="0.1" extlength="1" extoffset="8" precision="0" visible="yes"/>
+<dimension x1="91" y1="8" x2="96" y2="8" x3="93.5" y3="-9" textsize="1.27" layer="51" dtype="horizontal" extwidth="0.1" extlength="1" extoffset="8" precision="0" visible="yes"/>
+<dimension x1="96" y1="8" x2="101" y2="8" x3="98.5" y3="-9" textsize="1.27" layer="51" dtype="horizontal" extwidth="0.1" extlength="1" extoffset="8" precision="0" visible="yes"/>
+<dimension x1="101" y1="8" x2="106" y2="8" x3="103.5" y3="-9" textsize="1.27" layer="51" dtype="horizontal" extwidth="0.1" extlength="1" extoffset="8" precision="0" visible="yes"/>
+<dimension x1="50" y1="-10" x2="80" y2="-10" x3="65" y3="-7" textsize="1.27" layer="51" visible="yes"/>
+<dimension x1="0" y1="15" x2="0" y2="0" x3="-4" y3="7.5" textsize="1.27" layer="51" visible="yes"/>
+<dimension x1="0" y1="0" x2="50" y2="0" x3="25" y3="-7" textsize="1.27" layer="51" extoffset="3" visible="yes"/>
 </plain>
 <attributes>

Commit message: prettier schematics and BOM
Parts:
- C1, C21, C25, C6: value 10uF -> 10µF
- C13, C14, C15, C16, C18, C19, C2, C20, C26, C27, C5: value 0.1uF -> 0.1µF
- C17: value 10μF -> 10µF; device SparkFun:EIA3216 -> SparkFun-Capacitors:EIA3216
- C22: value 1u -> 1µF
- C33, C34, C35, C36, C9: value 1.0uF -> 1.0µF
- C37, C38: value 2.2uF -> 2.2µF
- renumbered JP1 to J1

Commit message: assembly drawings
Parts:
- added DRILEGEND: (no value), drilegend:DRILEGEND
- added U$1: (no value), frames:A4L-LOC
Other:
- board text added: "2.7.2016"
- board text added: "MP3 Player Marko Pero 2016"
- board text added: "v1.0"

Commit message: fixing missing wire on schematics
Connections:
- net PWM_LEFT: now also S5.P$1, S5.P$3
Changed lines of the file:
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@@
 <grid distance="1" unitdist="mm" unit="mm" style="lines" multiple="1" display="yes" altdistance="0.05" altunitdist="mm" altunit="mm"/>
 <layers>
-<layer number="1" name="Top" color="4" fill="1" visible="no" active="yes"/>
+<layer number="1" name="Top" color="4" fill="1" visible="yes" active="yes"/>
 <layer number="2" name="Route2" color="1" fill="3" visible="no" active="no"/>
 <layer number="3" name="Route3" color="4" fill="3" visible="no" active="no"/>
@@
 <layer number="14" name="Route14" color="1" fill="6" visible="no" active="no"/>
 <layer number="15" name="Route15" color="4" fill="6" visible="no" active="no"/>
-<layer number="16" name="Bottom" color="1" fill="1" visible="no" active="yes"/>
-<layer number="17" name="Pads" color="2" fill="1" visible="no" active="yes"/>
-<layer number="18" name="Vias" color="2" fill="1" visible="no" active="yes"/>
+<layer number="16" name="Bottom" color="1" fill="1" visible="yes" active="yes"/>
+<layer number="17" name="Pads" color="2" fill="1" visible="yes" active="yes"/>
+<layer number="18" name="Vias" color="2" fill="1" visible="yes" active="yes"/>
 <layer number="19" name="Unrouted" color="6" fill="1" visible="yes" active="yes"/>
 <layer number="20" name="Dimension" color="15" fill="1" visible="yes" active="yes"/>
@@
 <wire x1="173.228" y1="7.112" x2="173.4694" y2="7.042" width="0.254" layer="1"/>
 <via x="165.862" y="7.62" extent="1-16" drill="0.3"/>
+<contactref element="S5" pad="P$3"/>
+<contactref element="S5" pad="P$1"/>
+<wire x1="91.85" y1="6.4" x2="105.969" y2="7.118" width="0" layer="19" extent="1-16"/>
+<wire x1="91.85" y1="9.55" x2="91.85" y2="6.4" width="0" layer="19" extent="1-1"/>
 </signal>
 <signal name="N$29">

Commit message: Introduced to ATmega32u4 and redrew missing lines
Parts:
- removed U3: ATMEGA32U2, hf:TQFP32-08
- added U$3: ATMEGA32U4QFN2, SparkFun-DigitalIC:QFN-44-NOPAD
- OLED1: device microbuilder:UG-2832HSWEG04_WRAPAROUND -> pero_library:UG-2832HSWEG04
- Q1: value (none) -> 8MHz
- R11: device microbuilder:0805 -> rcl:R0603
Connections:
- removed net 3.3V2: R18.2, U3.6
- removed net N$11: U3.18
- removed net N$12: U3.7
- removed net N$30: U3.19
- removed net N$7: U3.13
- removed net SS: U3.14
- removed net VCC: C22.1, U3.27
- net 3.3V: now also C22.1, U$3.14, U$3.24, U$3.34, U$3.44, U$3.6; no longer U3.31, U3.32, U3.4
- net GND: now also J4.GND, U$3.15, U$3.23, U$3.35, U$3.43, U$3.5; no longer U3.28, U3.3
- net MISO: now also U$3.11; no longer U3.17
- net MOSI: now also U$3.10; no longer U3.16
- net N$1: now also R18.2, U$3.41; no longer U3.21
- net N$18: now also U$3.36; no longer U3.8
- net N$19: now also U$3.37; no longer U3.9
- net N$20: now also U$3.17; no longer U3.1
- net N$21: now also U$3.16; no longer U3.2
- net N$22: now also U$3.4; no longer U3.29
- net N$23: now also U$3.3; no longer U3.30
- net N$27: now also U$3.38; no longer U3.10
- net N$6: now also U$3.40; no longer U3.12
- net OLED-CS: now also U$3.26
- net OLED-DC: no longer U3.20
- net PWM_L: no longer U3.23
- net PWM_LEFT: now also U$3.39; no longer U3.11
- net PWM_R: no longer U3.25
- net RST: now also U$3.13; no longer U3.24
- net SCK: now also U$3.9; no longer U3.15
- net SD-CS: now also U$3.8
- net VUSB: now also U$3.7
Routing:
- net MOSI: track 154.1 -> 196.3 mm
- net 3.3V: track 368.9 -> 410.8 mm
- net N$22: track 29.7 -> 0.00 mm
- net N$23: track 25.2 -> 0.00 mm, vias 2 -> 0
- net N$45: track 8.35 -> 31.8 mm
- net N$44: track 5.07 -> 28.6 mm
- net N$55: track 11.6 -> 35.1 mm
- net N$48: track 10.7 -> 34.2 mm
- net N$47: track 5.65 -> 29.1 mm
- net N$49: track 15.8 -> 39.3 mm
- net N$46: track 20.7 -> 44.0 mm
- net OLED-DC: track 138.9 -> 162.1 mm
- net RST: track 16.5 -> 0.00 mm
- net 3.3V2: track 4.90 -> 0.00 mm
- net VCC: track 2.91 -> 0.00 mm
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Other:
- board text added: "27.9.2016"
- board text added: "v2.0"
- board text removed: "2.7.2016"
- board text removed: "v1.0"

Commit message: changed OLED footprint
Parts:
- moved OLED1 8.00 mm to (40.8, 7.65), flipped to the top
- moved R3 1.00 mm to (32.0, 10.0)
Connections:
- net MP3-CS: now also U$3.20
- net MP3-DCS: now also U$3.21
- net MP3-DREQ: now also U$3.18
- net MP3-RST: now also U$3.19
- net OLED-RST: now also U$3.25
- net PWM_L: now also U$3.30
- net PWM_R: now also U$3.29
Routing:
- net G1: track 4.86 -> 5.62 mm
Changed lines of the file:
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@@
 <layer number="20" name="Dimension" color="15" fill="1" visible="yes" active="yes"/>
 <layer number="21" name="tPlace" color="7" fill="1" visible="yes" active="yes"/>
-<layer number="22" name="bPlace" color="7" fill="1" visible="yes" active="yes"/>
+<layer number="22" name="bPlace" color="7" fill="1" visible="no" active="yes"/>
 <layer number="23" name="tOrigins" color="15" fill="1" visible="yes" active="yes"/>
-<layer number="24" name="bOrigins" color="15" fill="1" visible="yes" active="yes"/>
+<layer number="24" name="bOrigins" color="15" fill="1" visible="no" active="yes"/>
 <layer number="25" name="tNames" color="7" fill="1" visible="yes" active="yes"/>
 <layer number="26" name="bNames" color="7" fill="1" visible="no" active="yes"/>
-<layer number="27" name="tValues" color="7" fill="1" visible="no" active="yes"/>
+<layer number="27" name="tValues" color="7" fill="1" visible="yes" active="yes"/>
 <layer number="28" name="bValues" color="7" fill="1" visible="no" active="yes"/>
-<layer number="29" name="tStop" color="7" fill="3" visible="no" active="yes"/>
+<layer number="29" name="tStop" color="7" fill="3" visible="yes" active="yes"/>
 <layer number="30" name="bStop" color="7" fill="6" visible="no" active="yes"/>
-<layer number="31" name="tCream" color="7" fill="4" visible="yes" active="yes"/>
+<layer number="31" name="tCream" color="7" fill="4" visible="no" active="yes"/>
 <layer number="32" name="bCream" color="7" fill="5" visible="no" active="yes"/>
 <layer number="33" name="tFinish" color="6" fill="3" visible="no" active="yes"/>
@@
 <layer number="46" name="Milling" color="3" fill="1" visible="no" active="yes"/>
 <layer number="47" name="Measures" color="7" fill="1" visible="yes" active="yes"/>
-<layer number="48" name="Document" color="7" fill="1" visible="yes" active="yes"/>
+<layer number="48" name="Document" color="7" fill="1" visible="no" active="yes"/>
 <layer number="49" name="Reference" color="7" fill="1" visible="no" active="yes"/>
 <layer number="50" name="dxf" color="7" fill="1" visible="no" active="no"/>
-<layer number="51" name="tDocu" color="7" fill="1" visible="yes" active="yes"/>
-<layer number="52" name="bDocu" color="7" fill="1" visible="no" active="yes"/>
+<layer number="51" name="tDocu" color="7" fill="1" visible="no" active="yes"/>
+<layer number="52" name="bDocu" color="7" fill="1" visible="yes" active="yes"/>
 <layer number="53" name="tGND_GNDA" color="7" fill="9" visible="no" active="no"/>
 <layer number="54" name="bGND_GNDA" color="1" fill="9" visible="no" active="no"/>
@@
 <attribute name="VALUE" x="28.615" y="-0.905" size="1.27" layer="27"/>
 </element>
-<element name="R3" library="rcl" package="R0603" value="100k" x="32" y="11" smashed="yes" rot="MR0">
-<attribute name="NAME" x="31.785" y="11.835" size="1.27" layer="26" rot="MR0"/>
-<attribute name="VALUE" x="32.635" y="9.095" size="1.27" layer="28" rot="MR0"/>
+<element name="R3" library="rcl" package="R0603" value="100k" x="32" y="10" smashed="yes" rot="MR0">
+<attribute name="NAME" x="31.785" y="10.835" size="1.27" layer="26" rot="MR0"/>
+<attribute name="VALUE" x="32.635" y="8.095" size="1.27" layer="28" rot="MR0"/>
 </element>
 <element name="R4" library="rcl" package="R0603" value="100k" x="33" y="1" smashed="yes">
@@
 <attribute name="SUPPLIER-ID" value="SM02B-GHS-TB(LF)(SN)" x="189.049" y="9.954" size="1.778" layer="27" rot="R180" display="off"/>
 </element>
-<element name="OLED1" library="pero_library" package="UG-2832HSWEG04" value="UG-2832HSWEG04" x="48.8" y="7.652" smashed="yes" rot="MR0">
-<attribute name="NAME" x="84.4" y="11.852" size="1.27" layer="26" rot="MR0"/>
-<attribute name="VALUE" x="78.8" y="0.152" size="1.016" layer="28" rot="MR0"/>
+<element name="OLED1" library="pero_library" package="UG-2832HSWEG04" value="UG-2832HSWEG04" x="40.8" y="7.652" smashed="yes">
+<attribute name="NAME" x="5.2" y="11.852" size="1.27" layer="25"/>
+<attribute name="VALUE" x="10.8" y="0.152" size="1.016" layer="27"/>
 </element>
 <element name="C33" library="microbuilder" package="0805" value="1.0µF" x="62" y="5" smashed="yes">
@@
 <wire x1="61.05" y1="9" x2="61.05" y2="11" width="0" layer="19" extent="1-1"/>
 <wire x1="59.25" y1="7.5" x2="61.05" y2="9" width="0" layer="19" extent="1-1"/>
-<wire x1="33" y1="6.352" x2="59.25" y2="7.5" width="0" layer="19" extent="1-1"/>
+<wire x1="56.6" y1="6.352" x2="59.25" y2="7.5" width="0" layer="19" extent="1-1"/>
 <wire x1="56.45" y1="14.5" x2="61.15" y2="13" width="0" layer="19" extent="1-1"/>
 <wire x1="54" y1="12" x2="56.45" y2="14.5" width="0" layer="19" extent="1-1"/>
@@
 <wire x1="40" y1="2.25" x2="38.85" y2="1" width="0" layer="19" extent="1-1"/>
 <wire x1="38" y1="9.85" x2="37" y2="7.25" width="0" layer="19" extent="1-1"/>
-<wire x1="32.85" y1="11" x2="33.25" y2="11.25" width="0" layer="19" extent="1-16"/>
+<wire x1="32.85" y1="10" x2="33.25" y2="11.25" width="0" layer="19" extent="1-16"/>
 <wire x1="34.15" y1="11" x2="34.25" y2="10.25" width="0" layer="19" extent="1-16"/>
 <wire x1="33.875" y1="9.325" x2="34.25" y2="10.25" width="0" layer="19" extent="1-1"/>
 <wire x1="38" y1="11.85" x2="37.6" y2="10.25" width="0" layer="19" extent="1-16"/>
-<wire x1="31.5" y1="9.625" x2="32.85" y2="11" width="0" layer="19" extent="1-16"/>
+<wire x1="31.5" y1="9.625" x2="32.85" y2="10" width="0" layer="19" extent="1-16"/>
 <wire x1="27.75" y1="7.25" x2="27.75" y2="9.25" width="0" layer="19" extent="1-1"/>
 <wire x1="40.1" y1="11.85" x2="38" y2="11.85" width="0" layer="19" extent="16-16"/>
@@
 <wire x1="29.718" y1="10.668" x2="29.972" y2="10.922" width="0.254" layer="16"/>
 <wire x1="29.718" y1="12.192" x2="29.718" y2="10.668" width="0.254" layer="1"/>
-<wire x1="30.988" y1="10.922" x2="31.15" y2="11" width="0.254" layer="16"/>
+<wire x1="30.988" y1="10.922" x2="31.15" y2="10" width="0.254" layer="16"/>
 <wire x1="29.718" y1="12.192" x2="29.21" y2="12.192" width="0.254" layer="1"/>
 <wire x1="29.21" y1="12.192" x2="29.25" y2="12.25" width="0.254" layer="1"/>
@@
 <signal name="MP3-CS">
 <contactref element="U4" pad="23"/>
+<contactref element="U$3" pad="20"/>
+<wire x1="27.75" y1="5.75" x2="175.5" y2="9.4" width="0" layer="19" extent="1-1"/>
 </signal>
 <signal name="MP3-DCS">
 <contactref element="U4" pad="13"/>
+<contactref element="U$3" pad="21"/>
+<wire x1="27.75" y1="10.75" x2="175" y2="9.4" width="0" layer="19" extent="1-1"/>
 </signal>
 <signal name="MP3-RST">
@@
 <wire x1="36.1" y1="12.25" x2="37.5" y2="12.25" width="0.254" layer="1"/>
 <wire x1="37.5" y1="12.25" x2="39" y2="11" width="0.254" layer="1"/>
+<contactref element="U$3" pad="19"/>
+<wire x1="39" y1="11" x2="176" y2="9.4" width="0" layer="19" extent="1-1"/>
 </signal>
 <signal name="MP3-DREQ">
 <contactref element="U4" pad="8"/>
+<contactref element="U$3" pad="18"/>
+<wire x1="31.25" y1="12.25" x2="176.5" y2="9.4" width="0" layer="19" extent="1-1"/>
 </signal>
 <signal name="N$20">
@@
 <contactref element="OLED1" pad="8"/>
 <contactref element="U$3" pad="26"/>
-<wire x1="33" y1="7.652" x2="173.6" y2="7" width="0" layer="19" extent="1-1"/>
+<wire x1="56.6" y1="7.652" x2="173.6" y2="7" width="0" layer="19" extent="1-1"/>
 </signal>
 <signal name="OLED-RST">
 <contactref element="OLED1" pad="9"/>
+<contactref element="U$3" pad="25"/>
+<wire x1="56.6" y1="8.302" x2="173.6" y2="7.5" width="0" layer="19" extent="1-1"/>
 </signal>
 <signal name="OLED-DC">
@@
 <wire x1="27.866" y1="13.462" x2="27.588" y2="13.462" width="0.4064" layer="1"/>
 <wire x1="27.588" y1="13.462" x2="27.25" y2="13.8" width="0.4064" layer="1"/>
+<contactref element="U$3" pad="29"/>
+<wire x1="176.784" y1="5.842" x2="173.6" y2="5.5" width="0" layer="19" extent="1-16"/>
 </signal>
 <signal name="PWM_L">
@@
 <wire x1="6" y1="1" x2="174.228" y2="1" width="0.254" layer="16"/>
 <wire x1="174.228" y1="1" x2="176.276" y2="3.048" width="0.254" layer="16"/>
+<contactref element="U$3" pad="30"/>
+<wire x1="176.276" y1="3.048" x2="173.6" y2="5" width="0" layer="19" extent="1-16"/>
 </signal>
 <signal name="N$25">

Commit message: Autorouter dobar, al bez thermal pada
Parts:
- J1: value (none) -> Audio jack
- J4: value (none) -> micro USB
- moved C34 0.60 mm to (62.0, 6.40)
- moved C33 0.60 mm to (62.0, 4.40)
- moved C17 0.55 mm to (197.6, 7.62)
- moved C13 0.40 mm to (37.6, 9.00)
- moved C19 0.35 mm to (185.3, 8.48)
- moved C6 0.35 mm to (194.3, 2.92)
- moved C15 0.32 mm to (37.8, 1.25)
- moved R18 0.32 mm to (171.8, 11.7)
- moved Q1 0.25 mm to (181.0, 12.8)
- moved R4 0.22 mm to (32.9, 1.20)
- moved C18 0.15 mm to (172.0, 13.8)
- moved R2 0.15 mm to (29.2, 1.15)
- turned C2 to 180 degrees
- renumbered U$3 to U3
Connections:
- removed net N$29: OLED1.11
- net OLED-CS: now also U3.25; no longer U3.26
- net OLED-DC: now also U3.27
- net OLED-RST: now also U3.26; no longer U3.25
- net SCK: now also OLED1.11
Routing:
- net MP3-CS: track 0.00 -> 169.1 mm, vias 0 -> 2
- net MP3-DCS: track 0.00 -> 163.8 mm, vias 0 -> 6
- net MP3-DREQ: track 0.00 -> 160.1 mm
- net MP3-RST: track 8.85 -> 159.3 mm, vias 1 -> 7
- net OLED-RST: track 0.00 -> 131.8 mm, vias 0 -> 4
- net OLED-CS: track 0.00 -> 125.5 mm, vias 0 -> 6
- net 3.3V: track 410.8 -> 362.4 mm, vias 8 -> 20
- net PWM_LEFT: track 67.7 -> 108.1 mm, vias 1 -> 5
- net SD-CS: track 0.00 -> 39.4 mm, vias 0 -> 2
- net OLED-DC: track 162.1 -> 127.8 mm, vias 0 -> 6
- net N$22: track 0.00 -> 33.2 mm
- net N$46: track 44.0 -> 17.2 mm
- net N$48: track 34.2 -> 8.03 mm
- net N$49: track 39.3 -> 14.0 mm, vias 2 -> 0
- net N$45: track 31.8 -> 7.02 mm
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Other:
- outline, holes or cut-outs redrawn
