File: HW/MP3_Player.brd (EAGLE design)
At the start: 210 x 15 mm, 81 parts, among them J1 Audio jack, J2 LIPO-BATTERY-CONNECTOR, J3 USD-SDIO-SOCKETJLH, J4 micro USB, Q1 8MHz, Q2 12.288MHz, U1 3.3V/150mA, U2 1.8V/100mA, U3 ATMEGA32U4QFN2, U4 VS1053B, U5 MCP73831

Commit message: routing complete, no orphans
Routing:
- net GND: vias 16 -> 18
Changed lines of the file:
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@@
 <setting verticaltext="up"/>
 </settings>
-<grid distance="1" unitdist="mm" unit="mm" style="lines" multiple="1" display="yes" altdistance="0.05" altunitdist="mm" altunit="mm"/>
+<grid distance="39.3700787" unitdist="mil" unit="mil" style="lines" multiple="1" display="yes" altdistance="0.05" altunitdist="mm" altunit="mm"/>
 <layers>
 <layer number="1" name="Top" color="4" fill="1" visible="yes" active="yes"/>
@@
 <contactref element="S1" pad="P$3"/>
 <contactref element="LED2" pad="C"/>
-<polygon width="0.254" layer="16" orphans="yes">
+<polygon width="0.254" layer="16">
 <vertex x="0" y="15"/>
 <vertex x="210" y="15"/>
@@
 <vertex x="0" y="0"/>
 </polygon>
-<polygon width="0.254" layer="1" orphans="yes">
+<polygon width="0.254" layer="1">
 <vertex x="0" y="15"/>
 <vertex x="210" y="15"/>
@@
 <wire x1="33.6" y1="11.25" x2="33.3" y2="11.65" width="0.157" layer="1"/>
 <via x="34.15" y="10.35" extent="1-16" drill="0.3302"/>
+<via x="24.4" y="11.6" extent="1-16" drill="0.3302"/>
+<via x="26.085559375" y="9.45" extent="1-16" drill="0.3302"/>
 <wire x1="35.5092" y1="5.334" x2="34.25" y2="3.75" width="0" layer="19" extent="1-1"/>
-<wire x1="25.1" y1="11.85" x2="23.8" y2="12.3" width="0" layer="19" extent="1-16"/>
-<wire x1="27.75" y1="9.25" x2="27.75" y2="7.25" width="0" layer="19" extent="1-1"/>
-<wire x1="37.6" y1="9.85" x2="38" y2="11.85" width="0" layer="19" extent="1-16"/>
 <wire x1="147.21" y1="10.01" x2="147.21" y2="13.18" width="0" layer="19" extent="1-1"/>
 <wire x1="147.21" y1="2.96" x2="147.21" y2="10.01" width="0" layer="19" extent="1-1"/>
@@
 <wire x1="2.8956" y1="3.048" x2="2.85" y2="3" width="0.1524" layer="1"/>
 <wire x1="1.0668" y1="3.2004" x2="1" y2="3.1872" width="0.1524" layer="16"/>
-<wire x1="31.242" y1="7.7724" x2="36.1188" y2="7.7724" width="0.1524" layer="1"/>
-<wire x1="30.3276" y1="8.6868" x2="31.242" y2="7.7724" width="0.1524" layer="1"/>
+<wire x1="32" y1="7.7724" x2="36.1188" y2="7.7724" width="0.1524" layer="1"/>
 <wire x1="28.956" y1="10.0584" x2="30.3276" y2="8.6868" width="0.1524" layer="16"/>
 <wire x1="26.67" y1="10.0584" x2="28.956" y2="10.0584" width="0.1524" layer="16"/>
@@
 <wire x1="2.8956" y1="3.9624" x2="2.8956" y2="4.1148" width="0.1524" layer="1"/>
 <via x="2.8956" y="4.1148" extent="1-16" drill="0.3302"/>
-<via x="30.3276" y="8.6868" extent="1-16" drill="0.3302"/>
 <via x="26.67" y="10.0584" extent="1-16" drill="0.3302"/>
 <wire x1="25.7556" y1="10.9728" x2="26.67" y2="10.0584" width="0.1524" layer="1"/>
+<wire x1="30.3276" y1="8.6868" x2="30.8368" y2="8.6868" width="0.157" layer="16"/>
+<wire x1="30.8368" y1="8.6868" x2="30.85" y2="8.7" width="0.157" layer="16"/>
+<via x="30.85" y="8.7" extent="1-16" drill="0.3302"/>
+<wire x1="30.85" y1="8.7" x2="31.0724" y2="8.7" width="0.157" layer="1"/>
+<wire x1="31.0724" y1="8.7" x2="32" y2="7.7724" width="0.157" layer="1"/>
 </signal>
 <signal name="N$2">
@@
 <wire x1="35.3568" y1="9.144" x2="35.052" y2="9.144" width="0.1524" layer="1"/>
 <wire x1="29.1084" y1="8.0772" x2="28.6512" y2="8.0772" width="0.1524" layer="1"/>
-<wire x1="33.9852" y1="8.0772" x2="29.1084" y2="8.0772" width="0.1524" layer="16"/>
 <wire x1="35.052" y1="9.144" x2="33.9852" y2="8.0772" width="0.1524" layer="16"/>
 <wire x1="38.7096" y1="6.858" x2="38.5572" y2="6.858" width="0.1524" layer="1"/>
@@
 <wire x1="31.55" y1="2.4384" x2="32.004" y2="2.4384" width="0.157" layer="1"/>
 <wire x1="32.004" y1="2.4384" x2="32.6136" y2="3.048" width="0.157" layer="1"/>
+<wire x1="29.1084" y1="8.0772" x2="29.1728" y2="8.0772" width="0.157" layer="16"/>
+<wire x1="29.1728" y1="8.0772" x2="29.7" y2="7.55" width="0.157" layer="16"/>
+<wire x1="29.7" y1="7.55" x2="33.458" y2="7.55" width="0.157" layer="16"/>
+<wire x1="33.458" y1="7.55" x2="33.9852" y2="8.0772" width="0.157" layer="16"/>
 </signal>
 <signal name="1.8V">
@@
 <wire x1="27.8892" y1="5.1816" x2="27.75" y2="5.25" width="0.1524" layer="1"/>
 <wire x1="31.6992" y1="10.9728" x2="31.6992" y2="12.192" width="0.1524" layer="1"/>
-<wire x1="29.718" y1="8.9916" x2="31.6992" y2="10.9728" width="0.1524" layer="1"/>
-<wire x1="29.718" y1="5.1816" x2="29.718" y2="8.9916" width="0.1524" layer="1"/>
+<wire x1="30.1132" y1="9.3868" x2="31.6992" y2="10.9728" width="0.1524" layer="1"/>
 <wire x1="31.6992" y1="12.192" x2="31.75" y2="12.25" width="0.1524" layer="1"/>
 <wire x1="36.776" y1="4.8768" x2="43.5864" y2="4.8768" width="0.1524" layer="1"/>
@@
 <wire x1="43.434" y1="10.0584" x2="43.5864" y2="10.2108" width="0.157" layer="1"/>
 <wire x1="42.85" y1="11" x2="44.15" y2="11" width="0.157" layer="1"/>
+<wire x1="29.718" y1="5.1816" x2="29.718" y2="7.118" width="0.157" layer="1"/>
+<wire x1="29.718" y1="7.118" x2="30.1" y2="7.5" width="0.157" layer="1"/>
+<wire x1="30.1" y1="7.5" x2="30.1" y2="9.3736" width="0.157" layer="1"/>
+<wire x1="30.1" y1="9.3736" x2="30.1132" y2="9.3868" width="0.157" layer="1"/>
 </signal>
 <signal name="N$70">
