File: HW/MP3_Player.brd (EAGLE design)
At the start: 210 x 15 mm, 81 parts, among them J1 Audio jack, J2 LIPO-BATTERY-CONNECTOR, J3 USD-SDIO-SOCKETJLH, J4 micro USB, Q1 8MHz, Q2 12.288MHz, U1 3.3V/150mA, U2 1.8V/100mA, U3 ATMEGA32U4QFN2, U4 VS1053B, U5 MCP73831

Commit message: Autorouter finished
Parts:
- U3: value ATMEGA32U4QFN2 -> ATMEGA32U4QFN; device SparkFun-DigitalIC:QFN-44-NOPAD -> SparkFun-DigitalIC:QFN-44
Other:
- board text added: ">"
Changed lines of the file:
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@@
 <layer number="23" name="tOrigins" color="15" fill="1" visible="no" active="yes"/>
 <layer number="24" name="bOrigins" color="15" fill="1" visible="no" active="yes"/>
-<layer number="25" name="tNames" color="7" fill="1" visible="no" active="yes"/>
+<layer number="25" name="tNames" color="7" fill="1" visible="yes" active="yes"/>
 <layer number="26" name="bNames" color="7" fill="1" visible="no" active="yes"/>
 <layer number="27" name="tValues" color="7" fill="1" visible="no" active="yes"/>
@@
 <layer number="45" name="Holes" color="7" fill="1" visible="no" active="yes"/>
 <layer number="46" name="Milling" color="3" fill="1" visible="no" active="yes"/>
-<layer number="47" name="Measures" color="7" fill="1" visible="no" active="yes"/>
-<layer number="48" name="Document" color="7" fill="1" visible="no" active="yes"/>
-<layer number="49" name="Reference" color="7" fill="1" visible="no" active="yes"/>
+<layer number="47" name="Measures" color="7" fill="1" visible="yes" active="yes"/>
+<layer number="48" name="Document" color="7" fill="1" visible="yes" active="yes"/>
+<layer number="49" name="Reference" color="7" fill="1" visible="yes" active="yes"/>
 <layer number="50" name="dxf" color="7" fill="1" visible="no" active="no"/>
-<layer number="51" name="tDocu" color="7" fill="1" visible="no" active="yes"/>
+<layer number="51" name="tDocu" color="7" fill="1" visible="yes" active="yes"/>
 <layer number="52" name="bDocu" color="7" fill="1" visible="no" active="yes"/>
 <layer number="53" name="tGND_GNDA" color="7" fill="9" visible="no" active="no"/>
@@
 <layer number="131" name="tAdjust" color="7" fill="1" visible="no" active="yes"/>
 <layer number="132" name="bAdjust" color="7" fill="1" visible="no" active="yes"/>
-<layer number="144" name="DrillLegend" color="7" fill="1" visible="no" active="yes"/>
+<layer number="144" name="DrillLegend" color="7" fill="1" visible="yes" active="yes"/>
 <layer number="145" name="DrillLegend_01-16" color="2" fill="9" visible="no" active="yes"/>
 <layer number="146" name="DrillLegend_01-20" color="3" fill="9" visible="no" active="yes"/>
@@
 <wire x1="11.992" y1="8.492" x2="13.008" y2="8.492" width="0.1016" layer="146"/>
 <wire x1="13.008" y1="8.492" x2="11.992" y2="9.508" width="0.1016" layer="146"/>
+<text x="105.15" y="3.5" size="1.778" layer="21">&gt;</text>
 </plain>
 <attributes>
@@
 <element name="U$1" library="frames" package="A4L-LOC" value="" x="-29" y="-89"/>
 <element name="DRILEGEND" library="drilegend" package="DRILEGEND" value="" x="132.98400625" y="-24.826003125"/>
-<element name="U3" library="SparkFun-DigitalIC" package="QFN-44-NOPAD" value="ATMEGA32U4QFN2" x="177" y="6" rot="R180"/>
+<element name="U3" library="SparkFun-DigitalIC" package="QFN-44" value="ATMEGA32U4QFN" x="177" y="6" rot="R180"/>
 </elements>
 <signals>

Commit message: atmega routed
Parts:
- moved D2 0.50 mm to (203.0, 1.28)
- moved R17 0.40 mm to (185.3, 1.80)
- moved C11 0.25 mm to (10.8, 1.20)
Routing:
- net 3.3V: track 362.8 -> 294.2 mm, vias 20 -> 21
- net GBUF: track 41.7 -> 64.1 mm, vias 3 -> 5
- net MP3-CS: track 169.1 -> 185.7 mm, vias 2 -> 4
- net GND: track 16.1 -> 31.2 mm
- net MOSI: track 183.3 -> 198.4 mm, vias 7 -> 5
- net 1.8V: track 36.7 -> 50.6 mm, vias 3 -> 5
- net PWM_L: track 194.3 -> 181.2 mm
- net MISO: track 164.1 -> 175.9 mm, vias 10 -> 6
- net RIGHT: track 30.8 -> 19.7 mm
- net VIN: track 17.2 -> 26.1 mm
- net RST: track 16.1 -> 24.1 mm, vias 2 -> 4
- net N$1: track 21.9 -> 14.1 mm, vias 0 -> 2
- net N$22: track 33.2 -> 25.7 mm, vias 0 -> 2
- net PWM_R: track 161.7 -> 154.8 mm, vias 4 -> 6
- net SD-CS: track 39.4 -> 45.4 mm
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
Commit message: routed Oled
Routing:
- net OLED-RST: track 136.8 -> 139.0 mm
- net 3.3V: track 294.2 -> 295.5 mm
- net MOSI: track 198.4 -> 199.0 mm
- net GND: vias 18 -> 25

Commit message: passed DRC
Parts:
- moved C13 0.25 mm to (37.6, 8.75)
- moved Q1 0.16 mm to (180.9, 12.6)
- moved R4 0.11 mm to (32.9, 1.10)
Routing:
- net 3.3V: track 295.5 -> 300.5 mm
- net MOSI: track 199.0 -> 201.9 mm
- net GND: track 31.2 -> 34.1 mm, vias 25 -> 40
- net SCK: track 171.0 -> 173.2 mm
- net PWM_L: track 181.2 -> 179.2 mm
- net OLED-RST: track 139.0 -> 139.8 mm
- net MP3-DREQ: track 165.5 -> 166.2 mm
- net N$20: track 11.2 -> 11.8 mm
- net N$33: track 6.79 -> 7.38 mm
Other:
- outline, holes or cut-outs redrawn
