File: HW/MP3_Player.sch (EAGLE design)
At the start: 69 parts, among them IC3 ATMEGA8U2, J1 ISP/SPI, Q1 12.288MHz, U1 3.3V, U3 VS1053, U4 1.8V, U5 MCP73831, U6 USD-SOCKET, X2 USBSMD, Y2 8Mhz

Commit message: changed buttons, oscillator and JST connector
Parts:
- removed IC3: ATMEGA8U2, hf:ATMEGA8U2
- removed LCD3: UG-2832HSWEG04, microbuilder:OLED_UG-2832HSWEG04WRAPAROUND
- removed Y2: 8Mhz, SparkFun-FreqCtrl:CRYSTALSMD
- added C18, C19: 0.1uF, SparkFun-Capacitors:0.1UF-25V(+80/-20%)(0603)
- added C20: 0.1uF, rcl:C-EUC0603K
- added OLED1: UG-2832HSWEG04, microbuilder:OLED_UG-2832HSWEG04WRAPAROUND
- added Q2: 12.288MHz, SparkFun:CRYSTAL5X3
- added U2: 1.8V, SparkFun-PowerIC:V_REG_SP62141.8V
- C10, C11: device SparkFun-Capacitors:10NF/10000PF-50V-10%(0603) -> rcl:C-EUC0603K
- C12: device SparkFun-Capacitors:47NF(0.047UF/47000PF)-25V-5%(0603)SMD -> rcl:C-EUC0603K
- C13, C14, C15, C16, C2, C5: device SparkFun-Capacitors:0.1UF-25V(+80/-20%)(0603) -> rcl:C-EUC0603K
- C23, C24: value 20p -> 18p
- C3, C8: device SparkFun-Capacitors:22PF-50V-5%(0603) -> rcl:C-EUC0603K
- C4: device SparkFun-Capacitors:470PF-50V-5%(0603)SMD -> rcl:C-EUC0603K
- C7: device rcl:C-EUC0402 -> rcl:C-EUC0603K
- J2: value (none) -> LIPO-BATTERY-CONNECTOR; device SparkFun-Connectors:JST_2MM_MALE -> pero_library:LIPO-BATTERY-CONNECTOR
- Q1: value 12.288MHz -> (none); device SparkFun:CRYSTAL5X3 -> pero_library:QUARTZ-CRYSTAL-8MHZQC6CB8.00000F18B23R; PROD_ID XTAL-09653 -> (none)
- S1: value SWITCH-SMD -> Reset; device SparkFun:SWITCH-MOMENTARY-2SMD -> pero_library:SWITCH-BUTTON-SKSGAAE010
- S2: value PLAY/PAUSE -> Play/Pause; device SparkFun:SWITCH-MOMENTARY-2SMD -> pero_library:SWITCH-BUTTON-SKSGAAE010
- S3: device SparkFun:SWITCH-MOMENTARY-2SMD -> pero_library:SWITCH-BUTTON-SKSGAAE010
- S4: value BACK -> BCK; device SparkFun:SWITCH-MOMENTARY-2SMD -> pero_library:SWITCH-BUTTON-SKSGAAE010
- S5: value SWITCH-SMD -> SWITCH-BUTTON-SKSGAAE010; device SparkFun:SWITCH-MOMENTARY-2SMD -> pero_library:SWITCH-BUTTON-SKSGAAE010
- U3: value VS1053 -> ATMEGA32U2; device SparkFun-DigitalIC:VS1033/1053SMD -> hf:ATMEGA8U2
- U4: value 1.8V -> VS1053; device SparkFun-PowerIC:V_REG_SP62141.8V -> SparkFun-DigitalIC:VS1033/1053SMD
Connections:
- new net 3.3V1: C20.1
- new net OLED-DC: OLED1.D/C#, U3.(PCINT6)PB6
- net 1.8V: now also U2.OUT, U4.CVDD1, U4.CVDD2, U4.CVDD3, U4.CVDD4; no longer U3.CVDD1, U3.CVDD2, U3.CVDD3, U3.CVDD4, U4.OUT
- net 3.3V: now also C18.1, C19.1, OLED1.VBAT, OLED1.VDD, U2.EN, U2.IN, U3.AVCC, U3.UVCC, U3.VCC, U4.AVDD1, U4.AVDD2, U4.AVDD3, U4.IOVDD1, U4.IOVDD2, U4.IOVDD3, U4.TEST; no longer IC3.AVCC, IC3.UVCC, IC3.VCC, LCD3.VBAT, LCD3.VDD, U3.AVDD1, U3.AVDD2, U3.AVDD3, U3.IOVDD1, U3.IOVDD2, U3.IOVDD3, U3.TEST, U4.EN, U4.IN
- net G1: now also U4.GPIO2/DCLK, U4.GPIO3/SDATA, U4.GPIO6, U4.GPIO7; no longer U3.GPIO2/DCLK, U3.GPIO3/SDATA, U3.GPIO6, U3.GPIO7
- net G2: now also U4.GPIO5/I2C_MCLK; no longer U3.GPIO5/I2C_MCLK
- net GBUF: now also U4.GBUF; no longer U3.GBUF
- net GND: now also C18.2, C19.2, C20.2, OLED1.VSS, U2.GND, U3.GND, U3.UGND, U4.AGND1, U4.AGND2, U4.AGND3, U4.AGND4, U4.DGND1, U4.DGND2, U4.DGND3, U4.DGND4, U4.DGND5, U4.DGND6, U4.GPIO0/I2S_SCLK, U4.GPIO1/I2S_SDATA; no longer IC3.GND, IC3.UGND, LCD3.VSS, U3.AGND1, U3.AGND2, U3.AGND3, U3.AGND4, U3.DGND1, U3.DGND2, U3.DGND3, U3.DGND4, U3.DGND5, U3.DGND6, U3.GPIO0/I2S_SCLK, U3.GPIO1/I2S_SDATA, U4.GND
- net GPIO4: now also U4.GPIO4/I2S_LROUT; no longer U3.GPIO4/I2S_LROUT
- net LEFT: now also U4.LEFT; no longer U3.LEFT
- net MIDI-RX: now also U4.RX; no longer U3.RX
- net MISO: now also U3.(PDO/MISP/PCINT3)PB3, U4.S0; no longer IC3.(PDO/MISP/PCINT3)PB3, LCD3.D/C#, U3.S0
- net MOSI: now also OLED1.SDIN, U3.(PDI/MOSI/PCINT12)PB2, U4.SI; no longer IC3.(PDI/MOSI/PCINT12)PB2, LCD3.SDIN, U3.SI
- net MP3-CS: now also U4.XCS; no longer U3.XCS
- net MP3-DCS: now also U4.XDCS/BSYNC; no longer U3.XDCS/BSYNC
- net MP3-DREQ: now also U4.DREQ; no longer U3.DREQ
- net MP3-RST: now also U4.XRESET; no longer U3.XRESET
- net N$1: now also U3.(!RTS!/AIN5/INT6)PD6; no longer IC3.(!RTS!/AIN5/INT6)PD6
- net N$10: now also Q2.1, U4.XTAL2; no longer Q1.1, U3.XTAL2
- net N$11: now also U3.(T1/PCINT4)PB4; no longer IC3.(T1/PCINT4)PB4
- net N$12: now also U3.(RXD1/AIN1/INT2)PD2; no longer IC3.(RXD1/AIN1/INT2)PD2
- net N$18: now also U3.(PCINT10)PC4; no longer IC3.(PCINT11/AIN2)PC2
- net N$19: now also U3.(PCINT9/OC.1B)PC5; no longer IC3.(PCINT10)PC4
- net N$20: now also Q1.2, U3.XTAL1; no longer IC3.XTAL1, Y2.2
- net N$21: now also Q1.1, U3.XTAL2(PC0); no longer IC3.XTAL2(PC0), Y2.1
- net N$22: now also U3.D+; no longer IC3.D+
- net N$23: now also U3.D-; no longer IC3.D-
- net N$27: now also U3.(OC.1A/PCINT8)PC6; no longer IC3.(PCINT9/OC.1B)PC5
- net N$28: now also U3.(INT4/ICP1/CLK0)PC7; no longer IC3.(OC.1A/PCINT8)PC6
- net N$29: now also OLED1.SCLK; no longer LCD3.SCLK
- net N$30: now also U3.(PCINT5)PB5; no longer IC3.(PCINT5)PB5
- net N$44: now also OLED1.C2-; no longer LCD3.C2-
- net N$45: now also OLED1.C2+; no longer LCD3.C2+
- net N$46: now also OLED1.C1-; no longer LCD3.C1-
- net N$47: now also OLED1.C1+; no longer LCD3.C1+
- net N$48: now also OLED1.IREF; no longer LCD3.IREF
- net N$49: now also OLED1.VCOMH; no longer LCD3.VCOMH
- net N$55: now also OLED1.VCC; no longer LCD3.VCC
- net N$7: now also U3.(!HWB!/AIN6/T0/INT7)PD7; no longer IC3.(!HWB!/AIN6/T0/INT7)PD7
- net N$9: now also Q2.2, U4.XTAL1/MCLK; no longer Q1.2, U3.XTAL1/MCLK
- net OLED-CS: now also OLED1.CS#; no longer LCD3.CS#
- net OLED-RST: now also OLED1.RES#; no longer LCD3.RES#
- net RCAP: now also U4.RCAP; no longer U3.RCAP
- net RIGHT: now also U4.RIGHT; no longer U3.RIGHT
- net RST: now also U3.!RESET!(PC1/DW); no longer IC3.!RESET!(PC1/DW)
- net SCK: now also U3.(SCLK/PCINT1)PB1, U4.SCLK; no longer IC3.(SCLK/PCINT1)PB1, U3.SCLK
- net SS: now also U3.(!SS!/PCINT0)PB0; no longer IC3.(!SS!/PCINT0)PB0
- net VCC: now also U3.UCAP; no longer IC3.UCAP
Other:
- note added: "(Optional)"
- note added: "MP3 Decoder"
- note added: "uSD Interface"
- note removed: "VS1053"
- note removed: "microSD"
- moved on the sheet: C1, C10, C11, C12, C13, C14, C15, C16, C17, C2, C22, C23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

Commit message: Changed uSD socket. Components placed
Parts:
- removed LED3: Power, SparkFun:LED0603
- removed R12: 100k, SparkFun-Resistors:100KOHM1/10W1%(0603)
- removed R25: 1k, SparkFun:RESISTOR0402-RES
- removed U6: USD-SOCKET, SparkFun:USD-SOCKETNEW
- added C21, C25: (no value), SparkFun-Capacitors:CAP_POL1206
- added J3: USD-SDIO-SOCKETJLH, pero_library:USD-SDIO-SOCKETJLH
- added JP2, JP3, JP4: JUMPER-PAD-3-2OF3_NC_BY_TRACE_SMALL, SparkFun-Passives:JUMPER-PAD-3-2OF3_NC_BY_TRACE_SMALL
- added LED2: RED, SparkFun-LED:LED-RED0603
- added R18: 330, rcl:R-EU_R0603
- C10, C11, C12, C13, C14, C15, C20, C3, C4, C5, C8: device rcl:C-EUC0603K -> rcl:C-EUC0603
- C19: device SparkFun-Capacitors:0.1UF-25V(+80/-20%)(0603) -> rcl:C-EUC0603
- C9: device SparkFun-Capacitors:1.0UF-16V-10%(0603) -> rcl:C-EUC0603
- F2: value PTCSMD -> PTC0603; device SparkFun:PTCSMD -> SparkFun-PowerIC:PTC0603
- LED1: value Power -> RED
- R1: device SparkFun-Resistors:1M-1% -> rcl:R-EU_R0603
- R10, R14, R15, R16, R17: device SparkFun:RESISTOR0402-RES -> rcl:R-EU_R0603
- R2, R3, R4, R5: device SparkFun-Resistors:100KOHM1/10W1%(0603) -> rcl:R-EU_R0603
- R6, R7: device SparkFun-Resistors:20OHM1/10W1%(0603)SMD -> rcl:R-EU_R0603
- R8: device SparkFun-Resistors:330OHM1/10W1%(0603) -> rcl:R-EU_R0603
- R9: device SparkFun-Resistors:10OHM1/10W5%0603SMD -> rcl:R-EU_R0603
- S5: value SWITCH-BUTTON-SKSGAAE010 -> Reserved
- U1: value 3.3V -> 3.3V/150mA
- U2: value 1.8V -> 1.8V/100mA
- U4: value VS1053 -> VS1053B
Connections:
- net VBATT renamed VIN
- removed net 3.3V1: C20.1
- removed net D-1: R24.1
- removed net D-2: X2.D-
- removed net GPIO4: R12.2, U4.GPIO4/I2S_LROUT
- new net 3.3V2: R18.2, U3.(OC.0B/INT0)PD0
- new net N$17: R24.1, X2.D-
- new net PWM_L: C21.+, U3.(OC.1A/PCINT8)PC6
- new net PWM_LEFT: R16.2, S5.1, U3.(XCK_AIN4/PCINT12)PD5
- new net PWM_R: C25.+, U3.(PCINT9/OC.1B)PC5
- net 3.3V: now also C20.1, J3.VCC; no longer U6.VCC
- net G2: now also U4.GPIO0/I2S_SCLK, U4.GPIO1/I2S_SDATA, U4.GPIO4/I2S_LROUT
- net GBUF: now also JP4.1, JP4.2
- net GND: now also J3.CD1, J3.CD2, J3.GND, J3.SHIELD@1, J3.SHIELD@3, JP4.3, LED2.C; no longer LED3.C, R12.1, U4.GPIO0/I2S_SCLK, U4.GPIO1/I2S_SDATA, U6.GND, U6.SHIELD@1, U6.SHIELD@2, U6.SHIELD@3, U6.SHIELD@4
- net LEFT: now also JP2.1
- net MISO: now also J3.DAT0; no longer U6.DO
- net MOSI: now also J3.CMD; no longer U6.DI
- net N$12: now also U3.(AIN0/INT1)PD1; no longer U3.(RXD1/AIN1/INT2)PD2
- net N$14: now also JP2.2
- net N$18: now also U3.(RXD1/AIN1/INT2)PD2; no longer U3.(PCINT10)PC4
- net N$19: now also U3.(TXD1/INT3)PD3; no longer U3.(PCINT9/OC.1B)PC5
- net N$25: now also C21.-, JP2.3; no longer LED3.A, R25.1
- net N$27: now also U3.(INT5/AIN3)PD4; no longer U3.(OC.1A/PCINT8)PC6
- net N$28: now also C25.-, JP3.3; no longer R16.2, S5.1, U3.(INT4/ICP1/CLK0)PC7
- net N$8: now also LED2.A, R18.1; no longer C17.+, D2.A, U5.VIN
- net RIGHT: now also JP3.1, JP3.2
- net SCK: now also J3.CLK; no longer U6.SCK
- net SD-CS: now also J3.CD/DAT3; no longer U6.CS
- net VUSB: now also C17.+, D2.A, U5.VIN; no longer R25.2
Other:
- moved on the sheet: C10, C11, C12, C19, C20, F2, JP1, U4

Commit message: Micro USB instead of mini USB. Created "No MP3" variant. Audio jack verified.
Parts:
- removed X2: USBSMD, SparkFun:USBSMD
- added J4: (no value), SparkFun-Connectors:USB_MICROB_PLUGCONN-11752
Connections:
- net GND: no longer X2.GND
- net N$17: now also J4.D-; no longer X2.D-
- net N$24: now also J4.VCC; no longer X2.VBUS
- net N$26: now also J4.D+; no longer X2.D+
Changed lines of the file:
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@@
 </attributes>
 <variantdefs>
+<variantdef name="No MP3"/>
 </variantdefs>
 <classes>
@@
 <part name="LED1" library="SparkFun-LED" deviceset="LED-RED" device="0603" value="RED"/>
 <part name="GND7" library="SparkFun" deviceset="GND" device=""/>
-<part name="U4" library="SparkFun-DigitalIC" deviceset="VS1033/1053" device="SMD" value="VS1053B"/>
+<part name="U4" library="SparkFun-DigitalIC" deviceset="VS1033/1053" device="SMD" value="VS1053B">
+<variant name="No MP3" populate="no"/>
+</part>
 <part name="C1" library="SparkFun-Capacitors" deviceset="10UF-16V-10%(TANT)" device="" value="10uF"/>
 <part name="C2" library="rcl" deviceset="C-EU" device="C0603K" value="0.1uF"/>
-<part name="C3" library="rcl" deviceset="C-EU" device="C0603" value="22pF"/>
-<part name="C8" library="rcl" deviceset="C-EU" device="C0603" value="22pF"/>
+<part name="C3" library="rcl" deviceset="C-EU" device="C0603" value="22pF">
+<variant name="No MP3" populate="no"/>
+</part>
+<part name="C8" library="rcl" deviceset="C-EU" device="C0603" value="22pF">
+<variant name="No MP3" populate="no"/>
+</part>
 <part name="Q2" library="SparkFun" deviceset="CRYSTAL" device="5X3" value="12.288MHz">
 <attribute name="PROD_ID" value="XTAL-09653"/>
-</part>
-<part name="R1" library="rcl" deviceset="R-EU_" device="R0603" value="1M"/>
-<part name="C9" library="rcl" deviceset="C-EU" device="C0603" value="1.0uF"/>
-<part name="R2" library="rcl" deviceset="R-EU_" device="R0603" value="100k"/>
-<part name="R3" library="rcl" deviceset="R-EU_" device="R0603" value="100k"/>
-<part name="R5" library="rcl" deviceset="R-EU_" device="R0603" value="100k"/>
-<part name="R6" library="rcl" deviceset="R-EU_" device="R0603" value="20"/>
-<part name="R7" library="rcl" deviceset="R-EU_" device="R0603" value="20"/>
-<part name="R9" library="rcl" deviceset="R-EU_" device="R0603" value="10"/>
-<part name="C10" library="rcl" deviceset="C-EU" device="C0603" value="10nF"/>
-<part name="C11" library="rcl" deviceset="C-EU" device="C0603" value="10nF"/>
-<part name="C12" library="rcl" deviceset="C-EU" device="C0603" value="47nF"/>
+<variant name="No MP3" populate="no"/>
+</part>
+<part name="R1" library="rcl" deviceset="R-EU_" device="R0603" value="1M">
+<variant name="No MP3" populate="no"/>
+</part>
+<part name="C9" library="rcl" deviceset="C-EU" device="C0603" value="1.0uF">
+<variant name="No MP3" populate="no"/>
+</part>
+<part name="R2" library="rcl" deviceset="R-EU_" device="R0603" value="100k">
+<variant name="No MP3" populate="no"/>
+</part>
+<part name="R3" library="rcl" deviceset="R-EU_" device="R0603" value="100k">
+<variant name="No MP3" populate="no"/>
+</part>
+<part name="R5" library="rcl" deviceset="R-EU_" device="R0603" value="100k">
+<variant name="No MP3" populate="no"/>
+</part>
+<part name="R6" library="rcl" deviceset="R-EU_" device="R0603" value="20">
+<variant name="No MP3" populate="no"/>
+</part>
+<part name="R7" library="rcl" deviceset="R-EU_" device="R0603" value="20">
+<variant name="No MP3" populate="no"/>
+</part>
+<part name="R9" library="rcl" deviceset="R-EU_" device="R0603" value="10">
+<variant name="No MP3" populate="no"/>
+</part>
+<part name="C10" library="rcl" deviceset="C-EU" device="C0603" value="10nF">
+<variant name="No MP3" populate="no"/>
+</part>
+<part name="C11" library="rcl" deviceset="C-EU" device="C0603" value="10nF">
+<variant name="No MP3" populate="no"/>
+</part>
+<part name="C12" library="rcl" deviceset="C-EU" device="C0603" value="47nF">
+<variant name="No MP3" populate="no"/>
+</part>
 <part name="U2" library="SparkFun-PowerIC" deviceset="V_REG_SP6214" device="1.8V" value="1.8V/100mA"/>
 <part name="GND2" library="SparkFun" deviceset="GND" device=""/>
@@
 <part name="GND18" library="SparkFun" deviceset="GND" device=""/>
 <part name="C13" library="rcl" deviceset="C-EU" device="C0603" value="0.1uF"/>
-<part name="C14" library="rcl" deviceset="C-EU" device="C0603" value="0.1uF"/>
+<part name="C14" library="rcl" deviceset="C-EU" device="C0603" value="0.1uF">
+<variant name="No MP3" populate="no"/>
+</part>
 <part name="GND19" library="SparkFun" deviceset="GND" device=""/>
 <part name="GND20" library="SparkFun" deviceset="GND" device=""/>
-<part name="R4" library="rcl" deviceset="R-EU_" device="R0603" value="100k"/>
+<part name="R4" library="rcl" deviceset="R-EU_" device="R0603" value="100k">
+<variant name="No MP3" populate="no"/>
+</part>
 <part name="GND9" library="SparkFun" deviceset="GND" device=""/>
-<part name="C15" library="rcl" deviceset="C-EU" device="C0603" value="0.1uF"/>
+<part name="C15" library="rcl" deviceset="C-EU" device="C0603" value="0.1uF">
+<variant name="No MP3" populate="no"/>
+</part>
 <part name="GND23" library="SparkFun" deviceset="GND" device=""/>
 <part name="C16" library="rcl" deviceset="C-EU" device="C0603K" value="0.1uF"/>
@@
 <part name="GND42" library="supply1" deviceset="GND" device=""/>
 <part name="GND43" library="supply1" deviceset="GND" device=""/>
-<part name="X2" library="SparkFun" deviceset="USB" device="SMD"/>
 <part name="F2" library="SparkFun-PowerIC" deviceset="PTC" device="0603"/>
 <part name="GND44" library="SparkFun" deviceset="GND" device=""/>
@@
 <part name="P+11" library="SparkFun" deviceset="3.3V" device=""/>
 <part name="FRAME2" library="frames" deviceset="A3L-LOC" device=""/>
-<part name="C20" library="rcl" deviceset="C-EU" device="C0603" value="0.1uF"/>
+<part name="C20" library="rcl" deviceset="C-EU" device="C0603" value="0.1uF">
+<variant name="No MP3" populate="no"/>
+</part>
 <part name="GND31" library="SparkFun" deviceset="GND" device=""/>
 <part name="S1" library="pero_library" deviceset="SWITCH-BUTTON-SKSGAAE010" device="" value="Reset"/>
@@
 <part name="LED2" library="SparkFun-LED" deviceset="LED-RED" device="0603" value="RED"/>
 <part name="GND35" library="SparkFun" deviceset="GND" device=""/>
+<part name="J4" library="SparkFun-Connectors" deviceset="USB_MICROB_PLUG" device="CONN-11752"/>
 </parts>
 <sheets>
@@
 <instance part="GND42" gate="1" x="81.28" y="71.12"/>
 <instance part="GND43" gate="1" x="68.58" y="71.12"/>
-<instance part="X2" gate="G$1" x="22.86" y="104.14" rot="MR0"/>
 <instance part="F2" gate="G$1" x="38.1" y="106.68"/>
-<instance part="GND44" gate="1" x="27.94" y="99.06"/>
+<instance part="GND44" gate="1" x="35.56" y="116.84" rot="R90"/>
 <instance part="P+6" gate="G$1" x="78.74" y="144.78"/>
 <instance part="P+7" gate="G$1" x="81.28" y="124.46" smashed="yes">
@@
 <instance part="LED2" gate="G$1" x="187.96" y="63.5"/>
 <instance part="GND35" gate="1" x="187.96" y="53.34"/>
+<instance part="J4" gate="G$1" x="17.78" y="111.76" rot="R180"/>
 </instances>
 <busses>
@@
 </segment>
 <segment>
-<wire x1="25.4" y1="104.14" x2="27.94" y2="104.14" width="0.1524" layer="91"/>
-<wire x1="27.94" y1="104.14" x2="27.94" y2="101.6" width="0.1524" layer="91"/>
-<pinref part="X2" gate="G$1" pin="GND"/>
+<wire x1="25.4" y1="116.84" x2="33.02" y2="116.84" width="0.1524" layer="91"/>
 <pinref part="GND44" gate="1" pin="GND"/>
 </segment>
@@
 <segment>
 <wire x1="25.4" y1="106.68" x2="33.02" y2="106.68" width="0.1524" layer="91"/>
-<pinref part="X2" gate="G$1" pin="VBUS"/>
 <pinref part="F2" gate="G$1" pin="1"/>
+<pinref part="J4" gate="G$1" pin="VCC"/>
 </segment>
 </net>
 <net name="N$26" class="0">
 <segment>
-<pinref part="X2" gate="G$1" pin="D+"/>
 <pinref part="R23" gate="G$1" pin="1"/>
 <wire x1="25.4" y1="111.76" x2="63.5" y2="111.76" width="0.1524" layer="91"/>
+<pinref part="J4" gate="G$1" pin="D+"/>
 </segment>
 </net>
@@
 <net name="N$17" class="0">
 <segment>
-<pinref part="X2" gate="G$1" pin="D-"/>
 <pinref part="R24" gate="G$1" pin="1"/>
 <wire x1="25.4" y1="109.22" x2="53.34" y2="109.22" width="0.1524" layer="91"/>
+<pinref part="J4" gate="G$1" pin="D-"/>
 </segment>
 </net>
@@
 </sheet>
 </sheets>
+<errors>
+</errors>
 </schematic>
 </drawing>

Commit message: added 3d model. new button.
Parts:
- removed J1: ISP/SPI, SparkFun:AVR_SPI_PRG_6PTH
- removed LED1: RED, SparkFun-LED:LED-RED0603
- added S6: Vol Down, pero_library:SWITCH-BUTTON-SKSGAAE010
- C16, C2: device rcl:C-EUC0603K -> rcl:C-EUC0603
- C18: device SparkFun-Capacitors:0.1UF-25V(+80/-20%)(0603) -> rcl:C-EUC0603
- R8: value 330 -> 10k
- S5: value Reserved -> Vol Up
Connections:
- removed net 5V-MOSI: J1.4
- removed net 5V-SCK: J1.3
- net 3.3V: now also S6.2; no longer R8.2
- net GND: now also R8.1; no longer J1.6, LED1.C
- net MISO: no longer J1.1
- net N$1: now also U3.(PCINT7/OC.0A/OC.1C)PB7; no longer U3.(!RTS!/AIN5/INT6)PD6
- net N$6: now also R8.2, S6.1, U3.(!RTS!/AIN5/INT6)PD6; no longer LED1.A, R8.1
- net VCC: no longer J1.2
Other:
- moved on the sheet: C19, LED2, R18, R8

Commit message: Auto router not bad
Connections:
- net PWM_LEFT: no longer S5.1
Changed lines of the file:
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@@
 <setting verticaltext="up"/>
 </settings>
-<grid distance="0.1" unitdist="inch" unit="inch" style="lines" multiple="1" display="yes" altdistance="0.1" altunitdist="mm" altunit="mm"/>
+<grid distance="0.1" unitdist="inch" unit="inch" style="lines" multiple="1" display="no" altdistance="0.01" altunitdist="inch" altunit="inch"/>
 <layers>
 <layer number="1" name="Top" color="4" fill="1" visible="no" active="no"/>
@@
 <net name="PWM_LEFT" class="0">
 <segment>
-<pinref part="R16" gate="G$1" pin="2"/>
-<wire x1="177.8" y1="73.66" x2="177.8" y2="78.74" width="0.1524" layer="91"/>
-<pinref part="S5" gate="G$1" pin="1"/>
-<wire x1="177.8" y1="78.74" x2="177.8" y2="106.68" width="0.1524" layer="91"/>
 <pinref part="U3" gate="G$1" pin="(XCK_AIN4/PCINT12)PD5"/>
 <wire x1="142.24" y1="78.74" x2="177.8" y2="78.74" width="0.1524" layer="91"/>
-<junction x="177.8" y="78.74"/>
-</segment>
-</net>
+<pinref part="R16" gate="G$1" pin="2"/>
+<wire x1="177.8" y1="78.74" x2="177.8" y2="73.66" width="0.1524" layer="91"/>
+</segment>
+</net>

Commit message: Completed routing and verified. Added RC filters
Parts:
- added C26, C27: 0.1uF, rcl:C-EUC0603
- added R12, R19: 68, rcl:R-EU_R0603
- C21, C25: value (none) -> 10uF
Connections:
- net RCAP renamed N$33
- new net N$13: JP1.SLEEVE, JP4.2
- new net N$31: JP1.RIGHT, JP3.2
- new net N$32: C21.+, C26.1, R12.1
- new net PWM_L1: C25.+, C27.1, R19.1
- net GBUF: no longer JP1.SLEEVE, JP4.2
- net GND: now also C26.2, C27.2
- net PWM_L: now also R12.2; no longer C21.+
- net PWM_R: now also R19.2; no longer C25.+
- net RIGHT: no longer JP1.RIGHT, JP3.2
Other:
- moved on the sheet: C10, C11, C12, C25, C9, JP3, JP4, R6, R7, R9

Commit message: prettier schematics and BOM
Parts:
- C1, C6: value 10uF -> 10µF
- C13, C14, C15, C16, C18, C19, C2, C20, C26, C27, C5: value 0.1uF -> 0.1µF
- C17: value 10μF -> 10µF; device SparkFun:CAP_POL1206 -> SparkFun-Capacitors:10UF-16V-10%(TANT)
- C21, C25: value 10uF -> 10µF; device SparkFun-Capacitors:CAP_POL1206 -> SparkFun-Capacitors:10UF-16V-10%(TANT)
- C22: value 1u -> 1µF
- C33, C34, C35, C36, C9: value 1.0uF -> 1.0µF
- C37, C38: value 2.2uF -> 2.2µF
- R13: device rcl:R-US_R0603 -> rcl:R-EU_R0603
- renumbered JP1 to J1
