File: HW/MP3_Player.sch (EAGLE design)
At the start: 79 parts, among them J2 LIPO-BATTERY-CONNECTOR, J3 USD-SDIO-SOCKETJLH, Q2 12.288MHz, U1 3.3V/150mA, U2 1.8V/100mA, U3 ATMEGA32U2, U4 VS1053B, U5 MCP73831

Commit message: fixing missing wire on schematics
Connections:
- net PWM_LEFT: now also S5.1
Changed lines of the file:
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@@
 <pinref part="R16" gate="G$1" pin="2"/>
 <wire x1="177.8" y1="78.74" x2="177.8" y2="73.66" width="0.1524" layer="91"/>
+<pinref part="S5" gate="G$1" pin="1"/>
+<wire x1="177.8" y1="106.68" x2="177.8" y2="78.74" width="0.1524" layer="91"/>
+<junction x="177.8" y="78.74"/>
 </segment>
 </net>

Commit message: Introduced to ATmega32u4 and redrew missing lines
Parts:
- removed U3: ATMEGA32U2, hf:ATMEGA8U2
- added U$3: ATMEGA32U4QFN2, SparkFun-DigitalIC:ATMEGA32U4QFN2
- OLED1: device microbuilder:OLED_UG-2832HSWEG04WRAPAROUND -> pero_library:DISP_OLED_UG-2832HSWEG04
- Q1: value (none) -> 8MHz
- R11: device microbuilder:RESISTOR0805 -> rcl:R-EU_R0603
Connections:
- removed net 3.3V2: R18.2, U3.(OC.0B/INT0)PD0
- removed net N$11: U3.(T1/PCINT4)PB4
- removed net N$12: U3.(AIN0/INT1)PD1
- removed net N$30: U3.(PCINT5)PB5
- removed net N$7: U3.(!HWB!/AIN6/T0/INT7)PD7
- removed net SS: U3.(!SS!/PCINT0)PB0
- removed net VCC: C22.1, U3.UCAP
- net 3.3V: now also C22.1, U$3.AVCC@24, U$3.AVCC@44, U$3.UCAP, U$3.VCC@14, U$3.VCC@34; no longer U3.AVCC, U3.UVCC, U3.VCC
- net GND: now also J4.GND, U$3.GND@15, U$3.GND@23, U$3.GND@35, U$3.GND@43, U$3.UGND; no longer U3.GND, U3.UGND
- net MISO: now also U$3.PB3(MISO); no longer U3.(PDO/MISP/PCINT3)PB3
- net MOSI: now also U$3.PB2(MOSI); no longer U3.(PDI/MOSI/PCINT12)PB2
- net N$1: now also R18.2, U$3.PF0(ADC0); no longer U3.(PCINT7/OC.0A/OC.1C)PB7
- net N$18: now also U$3.PF7(ADC7); no longer U3.(RXD1/AIN1/INT2)PD2
- net N$19: now also U$3.PF6(ADC6); no longer U3.(TXD1/INT3)PD3
- net N$20: now also U$3.XTAL1; no longer U3.XTAL1
- net N$21: now also U$3.XTAL2; no longer U3.XTAL2(PC0)
- net N$22: now also U$3.D+; no longer U3.D+
- net N$23: now also U$3.D-; no longer U3.D-
- net N$27: now also U$3.PF5(ADC5); no longer U3.(INT5/AIN3)PD4
- net N$6: now also U$3.PF1(ADC1); no longer U3.(!RTS!/AIN5/INT6)PD6
- net OLED-CS: now also U$3.PD6(ADC9)
- net OLED-DC: no longer U3.(PCINT6)PB6
- net PWM_L: no longer U3.(OC.1A/PCINT8)PC6
- net PWM_LEFT: now also U$3.PF4(ADC4); no longer U3.(XCK_AIN4/PCINT12)PD5
- net PWM_R: no longer U3.(PCINT9/OC.1B)PC5
- net RST: now also U$3.!RESET; no longer U3.!RESET!(PC1/DW)
- net SCK: now also U$3.PB1(SCK); no longer U3.(SCLK/PCINT1)PB1
- net SD-CS: now also U$3.PB0(SS)
- net VUSB: now also U$3.VBUS
Other:
- note added: "v2.0"
- note removed: "v0.0"
- moved on the sheet: C18, C19, C22, C23, C24, F2, J4, LED2, Q1, R10, R14, R15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

Commit message: changed OLED footprint
Connections:
- net MP3-CS: now also U$3.PD2(RX)
- net MP3-DCS: now also U$3.PD3(TX)
- net MP3-DREQ: now also U$3.PD0(SCL)
- net MP3-RST: now also U$3.PD1(SDA)
- net OLED-RST: now also U$3.PD4(ADC8)
- net PWM_L: now also U$3.PB6(ADC13)
- net PWM_R: now also U$3.PB5(ADC12)
Changed lines of the file:
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@@
 </segment>
 <segment>
-<wire x1="124.46" y1="55.88" x2="132.08" y2="55.88" width="0.1524" layer="91"/>
 <pinref part="U$3" gate="G$1" pin="PB1(SCK)"/>
+<wire x1="132.08" y1="55.88" x2="124.46" y2="55.88" width="0.1524" layer="91"/>
 </segment>
 <segment>
@@
 </segment>
 <segment>
-<wire x1="124.46" y1="93.98" x2="132.08" y2="93.98" width="0.1524" layer="91"/>
+<pinref part="U$3" gate="G$1" pin="PD2(RX)"/>
+<wire x1="132.08" y1="93.98" x2="124.46" y2="93.98" width="0.1524" layer="91"/>
 </segment>
 </net>
@@
 </segment>
 <segment>
-<wire x1="127" y1="91.44" x2="132.08" y2="91.44" width="0.1524" layer="91"/>
-</segment>
-<segment>
-<wire x1="124.46" y1="91.44" x2="132.08" y2="91.44" width="0.1524" layer="91"/>
+<pinref part="U$3" gate="G$1" pin="PD3(TX)"/>
+<wire x1="132.08" y1="91.44" x2="124.46" y2="91.44" width="0.1524" layer="91"/>
 </segment>
 </net>
@@
 </segment>
 <segment>
-<wire x1="124.46" y1="88.9" x2="132.08" y2="88.9" width="0.1524" layer="91"/>
+<pinref part="U$3" gate="G$1" pin="PD1(SDA)"/>
+<wire x1="132.08" y1="88.9" x2="124.46" y2="88.9" width="0.1524" layer="91"/>
 </segment>
 </net>
@@
 </segment>
 <segment>
-<wire x1="124.46" y1="86.36" x2="132.08" y2="86.36" width="0.1524" layer="91"/>
-</segment>
-</net>
-<net name="SS" class="0">
-<segment>
-<wire x1="127" y1="58.42" x2="132.08" y2="58.42" width="0.1524" layer="91"/>
+<pinref part="U$3" gate="G$1" pin="PD0(SCL)"/>
+<wire x1="132.08" y1="86.36" x2="124.46" y2="86.36" width="0.1524" layer="91"/>
 </segment>
 </net>
@@
 </segment>
 <segment>
-<wire x1="124.46" y1="83.82" x2="132.08" y2="83.82" width="0.1524" layer="91"/>
+<pinref part="U$3" gate="G$1" pin="PD4(ADC8)"/>
+<wire x1="132.08" y1="83.82" x2="124.46" y2="83.82" width="0.1524" layer="91"/>
 </segment>
 </net>
@@
 <net name="PWM_R" class="0">
 <segment>
-<wire x1="124.46" y1="71.12" x2="132.08" y2="71.12" width="0.1524" layer="91"/>
 <label x="132.08" y="71.12" size="1.27" layer="95" xref="yes"/>
+<pinref part="U$3" gate="G$1" pin="PB5(ADC12)"/>
+<wire x1="132.08" y1="71.12" x2="124.46" y2="71.12" width="0.1524" layer="91"/>
 </segment>
 <segment>
@@
 <net name="PWM_L" class="0">
 <segment>
-<wire x1="124.46" y1="68.58" x2="132.08" y2="68.58" width="0.1524" layer="91"/>
 <label x="132.08" y="68.58" size="1.27" layer="95" xref="yes"/>
-</segment>
-<segment>
+<pinref part="U$3" gate="G$1" pin="PB6(ADC13)"/>
+<wire x1="132.08" y1="68.58" x2="124.46" y2="68.58" width="0.1524" layer="91"/>
+</segment>
+<segment>

Commit message: Autorouter dobar, al bez thermal pada
Parts:
- J1: value (none) -> Audio jack
- J4: value (none) -> micro USB
- renumbered U$3 to U3
Connections:
- removed net N$29: OLED1.SCLK
- net OLED-CS: now also U3.PD4(ADC8); no longer U3.PD6(ADC9)
- net OLED-DC: now also U3.PD7(ADC10)
- net OLED-RST: now also U3.PD6(ADC9); no longer U3.PD4(ADC8)
- net SCK: now also OLED1.SCLK

Commit message: Autorouter finished
Parts:
- U3: value ATMEGA32U4QFN2 -> ATMEGA32U4QFN; device SparkFun-DigitalIC:ATMEGA32U4QFN2 -> SparkFun-DigitalIC:ATMEGA32U4QFN
Changed lines of the file:
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@@
 <part name="C27" library="rcl" deviceset="C-EU" device="C0603" value="0.1µF"/>
 <part name="GND22" library="SparkFun" deviceset="GND" device=""/>
-<part name="U3" library="SparkFun-DigitalIC" deviceset="ATMEGA32U4" device="QFN2"/>
+<part name="U3" library="SparkFun-DigitalIC" deviceset="ATMEGA32U4" device="QFN" value="ATMEGA32U4QFN"/>
 <part name="GND34" library="supply1" deviceset="GND" device=""/>
 </parts>
