File: HW/MP3_Player.sch (EAGLE design)
At the start: 79 parts, among them J1 Audio jack, J2 LIPO-BATTERY-CONNECTOR, J3 USD-SDIO-SOCKETJLH, J4 micro USB, Q1 8MHz, Q2 12.288MHz, U1 3.3V/150mA, U2 1.8V/100mA, U3 ATMEGA32U4QFN, U4 VS1053B, U5 MCP73831

Commit message: First software version
Other:
- note added: "TO DO: _______________ * Change buttons to the pins with interrupt functions * No need forexternal pull up resistors, internal can be activated with PORTxn register"
Changed lines of the file:
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@@
 <?xml version="1.0" encoding="utf-8"?>
 <!DOCTYPE eagle SYSTEM "eagle.dtd">
-<eagle version="7.3.0">
+<eagle version="7.7.0">
 <drawing>
 <settings>
@@
 <text x="317.5" y="172.72" size="2.54" layer="97">OLED Interface</text>
 <text x="259.08" y="40.64" size="2.54" layer="97" ratio="15">(Optional)</text>
+<text x="25.4" y="142.24" size="1.778" layer="91">TO DO:
+_______________
+ * Change buttons to the pins with interrupt functions
+ * No need forexternal pull up resistors, internal can be activated with PORTxn register</text>
 </plain>
 <instances>
